File: Hardware/Audio_Filter.sch (KiCad schematic (older format))
At the start: 20 parts

Commit message: Added LED Strip Current Limiting Resistor
Added PSU surge protection caps
Parts:
- gave numbers to parts that had none: 20

Commit message: Annotated
Parts:
- renumbered C52 to C54, C53 to C55, C54 to C56, C55 to C57, C56 to C58, C57 to C59, C58 to C60, C59 to C61, R18 to R34, R19 to R35, R20 to R36, R21 to R37, R22 to R38, R23 to R39, R24 to R40, R25 to R41, R26 to R42

Commit message: Added Pull-down & Gate Resistors to MOSFETs
Parts:
- renumbered R34 to R58, R35 to R59, R36 to R60, R37 to R61, R38 to R62, R39 to R63, R40 to R64, R41 to R65, R42 to R66
Changed lines of the file:
@@
 	2950 3100 3200 3100
 $Comp
-L GND #PWR129
+L GND #PWR141
 U 1 1 57B0E099
 P 3150 3450
-AR Path="/57B136AF/57B0E099" Ref="#PWR129"  Part="1"
-AR Path="/57B0BDCC/57B0E099" Ref="#PWR139"  Part="1"
-F 0 "#PWR139" H 3150 3450 30  0001 C CNN
+AR Path="/57B136AF/57B0E099" Ref="#PWR141"  Part="1"
+AR Path="/57B0BDCC/57B0E099" Ref="#PWR151"  Part="1"
+F 0 "#PWR151" H 3150 3450 30  0001 C CNN
 F 1 "GND" H 3150 3380 30  0001 C CNN
 F 2 "" H 3150 3450 60  0000 C CNN
@@
 	3150 3300 3200 3300
 $Comp
-L +12V #PWR131
+L +12V #PWR143
 U 1 1 57B0E0A1
 P 3600 3950
-AR Path="/57B136AF/57B0E0A1" Ref="#PWR131"  Part="1"
-AR Path="/57B0BDCC/57B0E0A1" Ref="#PWR141"  Part="1"
-F 0 "#PWR141" H 3600 3900 20  0001 C CNN
+AR Path="/57B136AF/57B0E0A1" Ref="#PWR143"  Part="1"
+AR Path="/57B0BDCC/57B0E0A1" Ref="#PWR153"  Part="1"
+F 0 "#PWR153" H 3600 3900 20  0001 C CNN
 F 1 "+12V" H 3600 4050 30  0000 C CNN
 F 2 "" H 3600 3950 60  0000 C CNN
@@
 	3600 3950 3600 3600
 $Comp
-L -12V #PWR128
+L -12V #PWR140
 U 1 1 57B0E0A8
 P 3600 2700
-AR Path="/57B136AF/57B0E0A8" Ref="#PWR128"  Part="1"
-AR Path="/57B0BDCC/57B0E0A8" Ref="#PWR138"  Part="1"
-F 0 "#PWR138" H 3600 2830 20  0001 C CNN
+AR Path="/57B136AF/57B0E0A8" Ref="#PWR140"  Part="1"
+AR Path="/57B0BDCC/57B0E0A8" Ref="#PWR150"  Part="1"
+F 0 "#PWR150" H 3600 2830 20  0001 C CNN
 F 1 "-12V" H 3600 2800 30  0000 C CNN
 F 2 "" H 3600 2700 60  0000 C CNN
@@
 $EndComp
 $Comp
-L R R34
+L R R58
 U 1 1 57B0E0B6
 P 3700 2400
-AR Path="/57B136AF/57B0E0B6" Ref="R34"  Part="1"
-AR Path="/57B0BDCC/57B0E0B6" Ref="R43"  Part="1"
-F 0 "R43" V 3780 2400 40  0000 C CNN
+AR Path="/57B136AF/57B0E0B6" Ref="R58"  Part="1"
+AR Path="/57B0BDCC/57B0E0B6" Ref="R67"  Part="1"
+F 0 "R67" V 3780 2400 40  0000 C CNN
 F 1 "820" V 3707 2401 40  0000 C CNN
 F 2 "" V 3630 2400 30  0000 C CNN
@@
 	3000 5150 3200 5150
 $Comp
-L GND #PWR136
+L GND #PWR148
 U 1 1 57B0E0D2
 P 3150 5500
-AR Path="/57B136AF/57B0E0D2" Ref="#PWR136"  Part="1"
-AR Path="/57B0BDCC/57B0E0D2" Ref="#PWR146"  Part="1"
-F 0 "#PWR146" H 3150 5500 30  0001 C CNN
+AR Path="/57B136AF/57B0E0D2" Ref="#PWR148"  Part="1"
+AR Path="/57B0BDCC/57B0E0D2" Ref="#PWR158"  Part="1"
+F 0 "#PWR158" H 3150 5500 30  0001 C CNN
 F 1 "GND" H 3150 5430 30  0001 C CNN
 F 2 "" H 3150 5500 60  0000 C CNN
@@
 	3150 5350 3200 5350
 $Comp
-L +12V #PWR137
+L +12V #PWR149
 U 1 1 57B0E0DA
 P 3600 6000
-AR Path="/57B136AF/57B0E0DA" Ref="#PWR137"  Part="1"
-AR Path="/57B0BDCC/57B0E0DA" Ref="#PWR147"  Part="1"
-F 0 "#PWR147" H 3600 5950 20  0001 C CNN
+AR Path="/57B136AF/57B0E0DA" Ref="#PWR149"  Part="1"
+AR Path="/57B0BDCC/57B0E0DA" Ref="#PWR159"  Part="1"
+F 0 "#PWR159" H 3600 5950 20  0001 C CNN
 F 1 "+12V" H 3600 6100 30  0000 C CNN
 F 2 "" H 3600 6000 60  0000 C CNN
@@
 	3600 6000 3600 5650
 $Comp
-L -12V #PWR132
+L -12V #PWR144
 U 1 1 57B0E0E1
 P 3600 4750
-AR Path="/57B136AF/57B0E0E1" Ref="#PWR132"  Part="1"
-AR Path="/57B0BDCC/57B0E0E1" Ref="#PWR142"  Part="1"
-F 0 "#PWR142" H 3600 4880 20  0001 C CNN
+AR Path="/57B136AF/57B0E0E1" Ref="#PWR144"  Part="1"
+AR Path="/57B0BDCC/57B0E0E1" Ref="#PWR154"  Part="1"
+F 0 "#PWR154" H 3600 4880 20  0001 C CNN
 F 1 "-12V" H 3600 4850 30  0000 C CNN
 F 2 "" H 3600 4750 60  0000 C CNN
@@
 $EndComp
 $Comp
-L R R41
+L R R65
 U 1 1 57B0E0EF
 P 3700 4450
-AR Path="/57B136AF/57B0E0EF" Ref="R41"  Part="1"
-AR Path="/57B0BDCC/57B0E0EF" Ref="R50"  Part="1"
-F 0 "R50" V 3780 4450 40  0000 C CNN
+AR Path="/57B136AF/57B0E0EF" Ref="R65"  Part="1"
+AR Path="/57B0BDCC/57B0E0EF" Ref="R74"  Part="1"
+F 0 "R74" V 3780 4450 40  0000 C CNN
 F 1 "820" V 3707 4451 40  0000 C CNN
 F 2 "" V 3630 4450 30  0000 C CNN
@@
 Connection ~ 4300 4450
 $Comp
-L R R39
+L R R63
 U 1 1 57B0E101
 P 4850 4350
-AR Path="/57B136AF/57B0E101" Ref="R39"  Part="1"
-AR Path="/57B0BDCC/57B0E101" Ref="R48"  Part="1"
-F 0 "R48" V 4930 4350 40  0000 C CNN
+AR Path="/57B136AF/57B0E101" Ref="R63"  Part="1"
+AR Path="/57B0BDCC/57B0E101" Ref="R72"  Part="1"
+F 0 "R72" V 4930 4350 40  0000 C CNN
 F 1 "220" V 4857 4351 40  0000 C CNN
 F 2 "" V 4780 4350 30  0000 C CNN
@@
 $EndComp
 $Comp
-L R R36
+L R R60
 U 1 1 57B0E108
 P 4850 4150
-AR Path="/57B136AF/57B0E108" Ref="R36"  Part="1"
-AR Path="/57B0BDCC/57B0E108" Ref="R45"  Part="1"
-F 0 "R45" V 4930 4150 40  0000 C CNN
+AR Path="/57B136AF/57B0E108" Ref="R60"  Part="1"
+AR Path="/57B0BDCC/57B0E108" Ref="R69"  Part="1"
+F 0 "R69" V 4930 4150 40  0000 C CNN
 F 1 "220" V 4857 4151 40  0000 C CNN
 F 2 "" V 4780 4150 30  0000 C CNN
@@
 Connection ~ 5700 4150
 $Comp
-L R R37
+L R R61
 U 1 1 57B0E122
 P 6150 4150
-AR Path="/57B136AF/57B0E122" Ref="R37"  Part="1"
-AR Path="/57B0BDCC/57B0E122" Ref="R46"  Part="1"
-F 0 "R46" V 6230 4150 40  0000 C CNN
+AR Path="/57B136AF/57B0E122" Ref="R61"  Part="1"
+AR Path="/57B0BDCC/57B0E122" Ref="R70"  Part="1"
+F 0 "R70" V 6230 4150 40  0000 C CNN
 F 1 "180" V 6157 4151 40  0000 C CNN
 F 2 "" V 6080 4150 30  0000 C CNN
@@
 $EndComp
 $Comp
-L R R40
+L R R64
 U 1 1 57B0E129
 P 6150 4350
-AR Path="/57B136AF/57B0E129" Ref="R40"  Part="1"
-AR Path="/57B0BDCC/57B0E129" Ref="R49"  Part="1"
-F 0 "R49" V 6230 4350 40  0000 C CNN
+AR Path="/57B136AF/57B0E129" Ref="R64"  Part="1"
+AR Path="/57B0BDCC/57B0E129" Ref="R73"  Part="1"
+F 0 "R73" V 6230 4350 40  0000 C CNN
 F 1 "180" V 6157 4351 40  0000 C CNN
 F 2 "" V 6080 4350 30  0000 C CNN
@@
 	6400 4150 6600 4150
 $Comp
-L GND #PWR133
+L GND #PWR145
 U 1 1 57B0E132
 P 5850 5050
-AR Path="/57B136AF/57B0E132" Ref="#PWR133"  Part="1"
-AR Path="/57B0BDCC/57B0E132" Ref="#PWR143"  Part="1"
-F 0 "#PWR143" H 5850 5050 30  0001 C CNN
+AR Path="/57B136AF/57B0E132" Ref="#PWR145"  Part="1"
+AR Path="/57B0BDCC/57B0E132" Ref="#PWR155"  Part="1"
+F 0 "#PWR155" H 5850 5050 30  0001 C CNN
 F 1 "GND" H 5850 4980 30  0001 C CNN
 F 2 "" H 5850 5050 60  0000 C CNN
@@
 	7000 4650 7000 5050
 $Comp
-L R R42
+L R R66
 U 1 1 57B0E13A
 P 5850 4700
-AR Path="/57B136AF/57B0E13A" Ref="R42"  Part="1"
-AR Path="/57B0BDCC/57B0E13A" Ref="R51"  Part="1"
-F 0 "R51" V 5930 4700 40  0000 C CNN
+AR Path="/57B136AF/57B0E13A" Ref="R66"  Part="1"
+AR Path="/57B0BDCC/57B0E13A" Ref="R75"  Part="1"
+F 0 "R75" V 5930 4700 40  0000 C CNN
 F 1 "200" V 5857 4701 40  0000 C CNN
 F 2 "" V 5780 4700 30  0000 C CNN
@@
 	5850 4350 5850 4450
 $Comp
-L R R35
+L R R59
 U 1 1 57B0E143
 P 5850 3800
-AR Path="/57B136AF/57B0E143" Ref="R35"  Part="1"
-AR Path="/57B0BDCC/57B0E143" Ref="R44"  Part="1"
-F 0 "R44" V 5930 3800 40  0000 C CNN
+AR Path="/57B136AF/57B0E143" Ref="R59"  Part="1"
+AR Path="/57B0BDCC/57B0E143" Ref="R68"  Part="1"
+F 0 "R68" V 5930 3800 40  0000 C CNN
 F 1 "200" V 5857 3801 40  0000 C CNN
 F 2 "" V 5780 3800 30  0000 C CNN
@@
 Connection ~ 6500 4350
 $Comp
-L GND #PWR134
+L GND #PWR146
 U 1 1 57B0E15E
 P 6500 5050
-AR Path="/57B136AF/57B0E15E" Ref="#PWR134"  Part="1"
-AR Path="/57B0BDCC/57B0E15E" Ref="#PWR144"  Part="1"
-F 0 "#PWR144" H 6500 5050 30  0001 C CNN
+AR Path="/57B136AF/57B0E15E" Ref="#PWR146"  Part="1"
+AR Path="/57B0BDCC/57B0E15E" Ref="#PWR156"  Part="1"
+F 0 "#PWR156" H 6500 5050 30  0001 C CNN
 F 1 "GND" H 6500 4980 30  0001 C CNN
 F 2 "" H 6500 5050 60  0000 C CNN
@@
 $EndComp
 $Comp
-L +12V #PWR135
+L +12V #PWR147
 U 1 1 57B0E18D
 P 7000 5050
-AR Path="/57B136AF/57B0E18D" Ref="#PWR135"  Part="1"
-AR Path="/57B0BDCC/57B0E18D" Ref="#PWR145"  Part="1"
-F 0 "#PWR145" H 7000 5000 20  0001 C CNN
+AR Path="/57B136AF/57B0E18D" Ref="#PWR147"  Part="1"
+AR Path="/57B0BDCC/57B0E18D" Ref="#PWR157"  Part="1"
+F 0 "#PWR157" H 7000 5000 20  0001 C CNN
 F 1 "+12V" H 7000 5150 30  0000 C CNN
 F 2 "" H 7000 5050 60  0000 C CNN
@@
 $EndComp
 $Comp
-L -12V #PWR130
+L -12V #PWR142
 U 1 1 57B0E193
 P 7000 3750
-AR Path="/57B136AF/57B0E193" Ref="#PWR130"  Part="1"
-AR Path="/57B0BDCC/57B0E193" Ref="#PWR140"  Part="1"
-F 0 "#PWR140" H 7000 3880 20  0001 C CNN
+AR Path="/57B136AF/57B0E193" Ref="#PWR142"  Part="1"
+AR Path="/57B0BDCC/57B0E193" Ref="#PWR152"  Part="1"
+F 0 "#PWR152" H 7000 3880 20  0001 C CNN
 F 1 "-12V" H 7000 3850 30  0000 C CNN
 F 2 "" H 7000 3750 60  0000 C CNN
@@
 Connection ~ 6500 3450
 $Comp
-L R R38
+L R R62
 U 1 1 57B0E1AD
 P 8050 4250
-AR Path="/57B136AF/57B0E1AD" Ref="R38"  Part="1"
-AR Path="/57B0BDCC/57B0E1AD" Ref="R47"  Part="1"
-F 0 "R47" V 8130 4250 40  0000 C CNN
+AR Path="/57B136AF/57B0E1AD" Ref="R62"  Part="1"
+AR Path="/57B0BDCC/57B0E1AD" Ref="R71"  Part="1"
+F 0 "R71" V 8130 4250 40  0000 C CNN
 F 1 "100" V 8057 4251 40  0000 C CNN
 F 2 "" V 7980 4250 30  0000 C CNN

Commit message: Updated U8 reference location, Fixed Windows complaints
Parts:
- C54, C55, C56, C57, C58, C59, C60, C61: symbol C -> C-RESCUE-museV2
- R58, R59, R60, R61, R62, R63, R64, R65, R66: symbol R -> R-RESCUE-museV2
Changed lines of the file:
@@
 EESchema Schematic File Version 2
+LIBS:museV2-rescue
 LIBS:IntelEdisonBlockTemplate-cache
 LIBS:74xgxx
@@
 LIBS:microchip_pic18mcu
 LIBS:microchip
-LIBS:microchip1
 LIBS:microcontrollers
 LIBS:motorola
@@
 LIBS:sensors
 LIBS:siliconi
-LIBS:special
 LIBS:stm8
 LIBS:stm32
@@
 	2950 3100 3200 3100
 $Comp
-L GND #PWR141
+L GND-RESCUE-museV2 #PWR141
 U 1 1 57B0E099
 P 3150 3450
@@
 	3600 2700 3600 2800
 $Comp
-L C C54
+L C-RESCUE-museV2 C54
 U 1 1 57B0E0AF
 P 3700 2200
@@
 $EndComp
 $Comp
-L R R58
+L R-RESCUE-museV2 R58
 U 1 1 57B0E0B6
 P 3700 2400
@@
 Connection ~ 4300 2400
 $Comp
-L C C55
+L C-RESCUE-museV2 C55
 U 1 1 57B0E0C8
 P 3950 2600
@@
 	3000 5150 3200 5150
 $Comp
-L GND #PWR148
+L GND-RESCUE-museV2 #PWR148
 U 1 1 57B0E0D2
 P 3150 5500
@@
 	3600 4750 3600 4850
 $Comp
-L C C58
+L C-RESCUE-museV2 C58
 U 1 1 57B0E0E8
 P 3700 4250
@@
 $EndComp
 $Comp
-L R R65
+L R-RESCUE-museV2 R65
 U 1 1 57B0E0EF
 P 3700 4450
@@
 Connection ~ 4300 4450
 $Comp
-L R R63
+L R-RESCUE-museV2 R63
 U 1 1 57B0E101
 P 4850 4350
@@
 $EndComp
 $Comp
-L R R60
+L R-RESCUE-museV2 R60
 U 1 1 57B0E108
 P 4850 4150
@@
 	5100 4150 5900 4150
 $Comp
-L C C59
+L C-RESCUE-museV2 C59
 U 1 1 57B0E115
 P 5450 4250
@@
 Connection ~ 5700 4150
 $Comp
-L R R61
+L R-RESCUE-museV2 R61
 U 1 1 57B0E122
 P 6150 4150
@@
 $EndComp
 $Comp
-L R R64
+L R-RESCUE-museV2 R64
 U 1 1 57B0E129
 P 6150 4350
@@
 	6400 4150 6600 4150
 $Comp
-L GND #PWR145
+L GND-RESCUE-museV2 #PWR145
 U 1 1 57B0E132
 P 5850 5050
@@
 	7000 4650 7000 5050
 $Comp
-L R R66
+L R-RESCUE-museV2 R66
 U 1 1 57B0E13A
 P 5850 4700
@@
 	5850 4350 5850 4450
 $Comp
-L R R59
+L R-RESCUE-museV2 R59
 U 1 1 57B0E143
 P 5850 3800
@@
 Connection ~ 5850 4150
 $Comp
-L C C57
+L C-RESCUE-museV2 C57
 U 1 1 57B0E14C
 P 6500 3800
@@
 Connection ~ 6500 4150
 $Comp
-L C C61
+L C-RESCUE-museV2 C61
 U 1 1 57B0E155
 P 6500 4700
@@
 Connection ~ 6500 4350
 $Comp
-L GND #PWR146
+L GND-RESCUE-museV2 #PWR146
 U 1 1 57B0E15E
 P 6500 5050
@@
 	4200 2600 4150 2600
 $Comp
-L C C60
+L C-RESCUE-museV2 C60
 U 1 1 57B0E172
 P 3950 4650
@@
 	7000 3750 7000 3850
 $Comp
-L C C56
+L C-RESCUE-museV2 C56
 U 1 1 57B0E19A
 P 7350 3650
@@
 Connection ~ 6500 3450
 $Comp
-L R R62
+L R-RESCUE-museV2 R62
 U 1 1 57B0E1AD
 P 8050 4250
