File: Hardware/AUDIO_IO.sch (KiCad schematic (older format))
At the start: 10 parts

Commit message: Currently adding level shifters
Changed lines of the file:
@@
 LIBS:microchip_pic18mcu
 LIBS:microchip
+LIBS:microchip1
 LIBS:microcontrollers
 LIBS:motorola
@@
 LIBS:sensors
 LIBS:siliconi
+LIBS:special
 LIBS:stm8
 LIBS:stm32
@@
 Connection ~ 7650 2050
 Wire Wire Line
-	7650 1450 7650 2050
-Wire Wire Line
-	7650 2050 7650 2650
-Wire Wire Line
-	7650 2650 7650 3250
-Wire Wire Line
-	7650 3250 7650 3450
+	7650 1450 7650 3450
 Wire Wire Line
 	7350 1450 7650 1450
@@
 	3200 3500 3300 3500
 Wire Wire Line
-	3200 3600 3200 3700
-Wire Wire Line
-	3200 3700 3200 3900
+	3200 3600 3200 3900
 Wire Wire Line
 	3200 3600 3300 3600
@@
 	3100 4700 3650 4700
 Wire Wire Line
-	4750 4600 4750 4700
-Wire Wire Line
-	4750 4700 4750 4900
+	4750 4600 4750 4900
 Wire Wire Line
 	4750 4600 4650 4600
