File: Hardware/museV2.sch (KiCad schematic (older format))
At the start: 164 parts, among them J1 ATX24, J2 ATX24, P1 RCA_Stero_Jack, P10 AI_RGB, P11 CONN_01X04, P12 AI_RGB, P13 AI_RGB, P14 AI_RGB, P15 AI_RGB, P16 CONN_01X04, P17 AI_RGB, P18 AI_RGB, P19 AI_RGB, P2 CONN_01X06, P20 AI_RGB, P21 AI_RGB, P22 CONN_01X04, P23 AI_RGB, P24 AI_RGB, P25 AI_RGB, P3 3.5mm_Audio, P4 RCA_Stero_Jack, P5 3.5mm_Audio, P6 CONN_01X04, P7 AI_RGB, P8 AI_RGB, P9 AI_RGB, Q1 MOSFET_N, Q10 MOSFET_N, Q11 MOSFET_N, Q12 MOSFET_N, Q13 MOSFET_N, Q2 MOSFET_N, Q3 MOSFET_N, Q4 MOSFET_N, Q5 MOSFET_N, Q6 MOSFET_N, Q7 BSS138, Q8 MOSFET_N, Q9 MOSFET_N, SW1 PWR_BTN, U1 POM-3535L-3-R, U10 PCM1863, U11 PCM1796, U2 PLR135/T10, U3 POM-3535L-3-R, U4 PLT133/T10W, U5 POM-3535L-3-R, U6 POM-3535L-3-R, U7 PCM9211, U8 EdisonConnector, U9 LP38692, X1 24.576 MHz

Commit message: Added level shifter, moved LEDs to their own sheet
Parts:
- removed P10, P12, P13, P14, P15, P17, P18, P19, P20, P21, P23, P24, P25, P7, P8, P9: AI_RGB, symbol CONN_01X03
- removed P11, P16, P22, P6: CONN_01X04, symbol CONN_01X04
- removed Q1, Q10, Q11, Q12, Q13, Q2, Q3, Q4, Q5, Q6, Q8, Q9: MOSFET_N, symbol MOSFET_N
- removed R1, R12, R13, R18, R26, R27, R29, R3, R40, R42, R43, R5: 100, symbol R-RESCUE-museV2
- removed R10, R11, R15, R19, R2, R24, R25, R28, R30, R34, R35, R4, R41, R44, R48, R9: 470, symbol R-RESCUE-museV2
- removed R20, R21, R22, R31, R32, R33, R45, R46, R47, R6, R7, R8: 1M, symbol R-RESCUE-museV2
- added U?: GTL2010, symbol GTL2010
Connections:
- wire segments 746 -> 481
- no-connect marks 45 -> 44
Other:
- note added: "LED Light Connections"
- note removed: "Individually \nAddressable\nRGB LED Strips"
- note removed: "Single RGB LED Strips"
- moved on the sheet: C35, C36

Commit message: Added PWM generator, More Shift Regs
Moved GPIO pins on MUSE
Parts:
- added R?: 220, symbol R-RESCUE-museV2
- added U?: GTL2010, symbol GTL2010
Connections:
- net labels added: ADC_ESEN_INT(1.8), DFE_RST(1.8), EDI_RST_OUT(1.8), I2C_SCA(1.8), I2C_SCL(1.8), I2S_MCU_BCK(1.8), I2S_MCU_DIN(1.8), I2S_MCU_DOUT(1.8), I2S_MCU_LRCK(1.8), I2S_SCK(1.8), LED_IA_1(1.8), LED_IA_10(1.8), LED_IA_11(1.8), LED_IA_12(1.8), LED_IA_13(1.8), LED_IA_14(1.8), LED_IA_15(1.8), LED_IA_16(1.8), LED_IA_2(1.8), LED_IA_3(1.8), LED_IA_4(1.8), LED_IA_5(1.8), LED_IA_6(1.8), LED_IA_7(1.8), LED_IA_8(1.8), LED_IA_9(1.8), LED_PWM_SCL, LED_PWM_SCL(1.8), LED_PWM_SDA, LED_PWM_SDA(1.8), UART_RX(1.8), UART_TX(1.8), ~LED_PWM_OE
- net labels removed: EDI_RST_OUT, I2C_SCA, LED_B_1, LED_B_2, LED_B_3, LED_B_4, LED_G_1, LED_G_2, LED_G_3, LED_G_4, LED_R_1, LED_R_2, LED_R_3, LED_R_4, SPDIF_LOCK
- wire segments 481 -> 477
- no-connect marks 44 -> 40
Other:
- note added: "From \nMCU(Control)"
- note added: "I2C Addr 0x80/0x81"
- note added: "Pulled LOW for\nI2C mode Addr 0x94"
- note added: "To DFE\n(Bluetooth/\nAnalog input)"
- note removed: "From MCU\n(Control)"
- moved on the sheet: C47, R14, R16, SW1, U8, U?

Commit message: Syncing changes from 9/20 meeting
Parts:
- removed C35, C36: 1uF, symbol C-RESCUE-museV2
- removed D1: PWR_LED, symbol LED-RESCUE-museV2
- removed J1, J2: ATX24, symbol ATX24
- removed P1, P4: RCA_Stero_Jack, symbol RCA_Stero_Jack
- removed P3, P5: 3.5mm_Audio, symbol CONN_01X03
- removed Q7: BSS138, SOT-23, symbol BSS138
- removed R14, R16: 10K, symbol R-RESCUE-museV2
- removed R17: 576, symbol R-RESCUE-museV2
- removed R?: 220, symbol R-RESCUE-museV2
- removed SW1: PWR_BTN, symbol SW_PUSH
- removed U1, U3, U5, U6: POM-3535L-3-R, symbol POM-3535L-3-R
- removed U2: PLR135/T10, symbol PLR135/10
- removed U4: PLT133/T10W, symbol PLT133/T10W
- removed U9: LP38692, symbol LP38692
- removed U? (x2): GTL2010, symbol GTL2010
Connections:
- net labels added: I2C_PWM_SCL, I2C_PWM_SCL(1.8), I2C_PWM_SDA, I2C_PWM_SDA(1.8)
- net labels removed: +12V_AUX, +5V_AUX, -5V, ADC_ESEN_INT(1.8), ATX_PS_OK, AUX_PS_OK, DFE_RST(1.8), EDISON_PWR_BTN, EDISON_RST_OUT, I2S_SCK(1.8), LED_PWM_SCL, LED_PWM_SCL(1.8), LED_PWM_SDA, LED_PWM_SDA(1.8), ~LED_PWM_OE
- wire segments 477 -> 459
- no-connect marks 40 -> 45
Other:
- note added: "To LED\nPWM\ngenerator"
- note removed: "5VSB->3.3VSB LDO"
- note removed: "ATX Power Connectors"
- note removed: "Analog Audio Connections"
- note removed: "Digital Audio (S/PDIF) Connections"
- note removed: "Intel Edison Power Control"
- note removed: "Microphones"
- note removed: "Optical In"
- note removed: "Optical Output"
- note removed: "To DFE\n(Bluetooth/\nAnalog input)"
- moved on the sheet: P2

Commit message: Currently adding level shifters
Connections:
- wire segments 459 -> 362

Commit message: Finished level shifter sheet
Connections:
- net Audio_Filter/ANALOG_OUT+ is gone; now on net Audio_Filter/ANALOG_OUT+: U11.25 (IOUT_L+)
- net Audio_Filter/ANALOG_OUT- is gone; now on net Audio_Filter/ANALOG_OUT-: U11.26 (IOUT_L-)
- net Audio_Filter/ANALOG_OUT+: no longer U11.17 (IOUT_R+)
- net Audio_Filter/ANALOG_OUT-: no longer U11.18 (IOUT_R-)
- new net Audio_Filter/ANALOG_OUT+: U11.17 (IOUT_R+)
- new net Audio_Filter/ANALOG_OUT-: U11.18 (IOUT_R-)
Changed lines of the file:
@@
 $EndComp
 $Sheet
-S 14750 3300 850  2200
+S 14750 3300 950  2200
 U 57E226F1
 F0 "LIGHT_CONN" 60
@@
 I2C_PWM_SCL(1.8)
 $Sheet
-S 13550 6500 900  3200
+S 13750 6500 950  2800
 U 57E80EBA
 F0 "LEVEL_SHIFTER" 60
 F1 "LEVEL_SHIFTER.sch" 60
-F2 "1(1.8)" I L 13550 6600 60
-F3 "2(1.8)" I L 13550 6700 60
-F4 "3(1.8)" I L 13550 6800 60
-F5 "4(1.8)" I L 13550 6900 60
-F6 "5(1.8)" I L 13550 7000 60
-F7 "6(1.8)" I L 13550 7100 60
-F8 "7(1.8)" I L 13550 7200 60
-F9 "8(1.8)" I L 13550 7300 60
-F10 "9(1.8)" I L 13550 7400 60
-F11 "10(1.8)" I L 13550 7500 60
-F12 "11(1.8)" I L 13550 7650 60
-F13 "12(1.8)" I L 13550 7750 60
-F14 "13(1.8)" I L 13550 7850 60
-F15 "14(1.8)" I L 13550 7950 60
-F16 "15(1.8)" I L 13550 8050 60
-F17 "16(1.8)" I L 13550 8150 60
-F18 "17(1.8)" I L 13550 8250 60
-F19 "18(1.8)" I L 13550 8350 60
-F20 "19(1.8)" I L 13550 8450 60
-F21 "20(1.8)" I L 13550 8550 60
-F22 "21(1.8)" I L 13550 8700 60
-F23 "22(1.8)" I L 13550 8800 60
-F24 "23(1.8)" I L 13550 8900 60
-F25 "24(1.8)" I L 13550 9000 60
-F26 "25(1.8)" I L 13550 9100 60
-F27 "26(1.8)" I L 13550 9200 60
-F28 "27(1.8)" I L 13550 9300 60
-F29 "28(1.8)" I L 13550 9400 60
-F30 "29(1.8)" I L 13550 9500 60
-F31 "30(1.8)" I L 13550 9600 60
+F2 "1(1.8)" I L 13750 6600 60
+F3 "2(1.8)" I L 13750 6700 60
+F4 "3(1.8)" I L 13750 6800 60
+F5 "4(1.8)" I L 13750 6900 60
+F6 "5(1.8)" I L 13750 7000 60
+F7 "6(1.8)" I L 13750 7100 60
+F8 "7(1.8)" I L 13750 7200 60
+F9 "8(1.8)" I L 13750 7300 60
+F10 "9(1.8)" I L 13750 7400 60
+F11 "10(1.8)" I L 13750 7500 60
+F12 "11(1.8)" I L 13750 7650 60
+F13 "12(1.8)" I L 13750 7750 60
+F14 "13(1.8)" I L 13750 7850 60
+F15 "14(1.8)" I L 13750 7950 60
+F16 "15(1.8)" I L 13750 8050 60
+F17 "16(1.8)" I L 13750 8150 60
+F18 "17(1.8)" I L 13750 8250 60
+F19 "18(1.8)" I L 13750 8350 60
+F20 "19(1.8)" I L 13750 8450 60
+F21 "20(1.8)" I L 13750 8550 60
+F22 "21(1.8)" I L 13750 8700 60
+F23 "22(1.8)" I L 13750 8800 60
+F24 "23(1.8)" I L 13750 8900 60
+F25 "24(1.8)" I L 13750 9000 60
+F26 "25(1.8)" I L 13750 9100 60
+F27 "26(1.8)" I L 13750 9200 60
+F28 "1(3.3)" I R 14700 6600 60
+F29 "2(3.3)" I R 14700 6700 60
+F30 "3(3.3)" I R 14700 6800 60
+F31 "4(3.3)" I R 14700 6900 60
+F32 "5(3.3)" I R 14700 7000 60
+F33 "6(3.3)" I R 14700 7100 60
+F34 "7(3.3)" I R 14700 7200 60
+F35 "8(3.3)" I R 14700 7300 60
+F36 "9(3.3)" I R 14700 7400 60
+F37 "10(3.3)" I R 14700 7500 60
+F38 "1(5.0)" I R 14700 7650 60
+F39 "2(5.0)" I R 14700 7750 60
+F40 "3(5.0)" I R 14700 7850 60
+F41 "4(5.0)" I R 14700 7950 60
+F42 "5(5.0)" I R 14700 8050 60
+F43 "6(5.0)" I R 14700 8150 60
+F44 "7(5.0)" I R 14700 8250 60
+F45 "8(5.0)" I R 14700 8350 60
+F46 "9(5.0)" I R 14700 8450 60
+F47 "10(5.0)" I R 14700 8550 60
+F48 "11(5.0)" I R 14700 8700 60
+F49 "12(5.0)" I R 14700 8800 60
+F50 "13(5.0)" I R 14700 8900 60
+F51 "14(5.0)" I R 14700 9000 60
+F52 "15(5.0)" I R 14700 9100 60
+F53 "16(5.0)" I R 14700 9200 60
 $EndSheet
 Text Notes 11650 7600 0    60   ~ 0

Commit message: In progress changing to global labels
Connections:
- net Audio_Filter/ANALOG_OUT+ is gone; now on net Audio_Filter/ANALOG_OUT+: U11.25 (IOUT_L+)
- net Audio_Filter/ANALOG_OUT- is gone; now on net Audio_Filter/ANALOG_OUT-: U11.26 (IOUT_L-)
- net Audio_Filter/ANALOG_OUT+: no longer U11.17 (IOUT_R+)
- net Audio_Filter/ANALOG_OUT-: no longer U11.18 (IOUT_R-)
- net I2S_MCU_BCK: no longer U7.30 (RXIN5/ABCKI0)
- net I2S_MCU_LRCK: no longer U7.29 (RXIN6/ALRCKI0)
- net I2S_SCK: no longer U7.31 (RXIN4/ASCKI0)
- net I2C_SCL renamed I2C_SCL(3.3)
- net I2C_SDA renamed I2C_SDA(3.3)
- net I2S_MCU_DOUT renamed I2S_MCU_DOUT(3.3)
- net UART_RX renamed UART_RX(3.3)
- net UART_TX renamed UART_TX(3.3)
- new net Audio_Filter/ANALOG_OUT+: U11.17 (IOUT_R+)
- new net Audio_Filter/ANALOG_OUT-: U11.18 (IOUT_R-)
- new net I2S_MCU_BCK(3.3): U7.30 (RXIN5/ABCKI0)
- new net I2S_MCU_LRCK(3.3): U7.29 (RXIN6/ALRCKI0)
- new net I2S_SCK(3.3): U7.31 (RXIN4/ASCKI0)
Other:
- moved on the sheet: C37, C38, C39, C40, C41, C42, C43, C44, C45, C46, C48, C49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

Commit message: Changing to global labels/pages in progress
Parts:
- removed C37, C42: 27pF, symbol C-RESCUE-museV2
- removed C38, C52: 0.1uF, symbol C-RESCUE-museV2
- removed C39, C43, C44, C45, C46, C48, C49, C50, C51: 10uF, symbol C-RESCUE-museV2
- removed C40: .068uF, symbol C-RESCUE-museV2
- removed C41: 4700pF, symbol C-RESCUE-museV2
- removed C53: 1uF, symbol C-RESCUE-museV2
- removed R23: 680, symbol R-RESCUE-museV2
- removed R36, R37, R38, R39, R50, R51, R52, R53: 100K, symbol R-RESCUE-museV2
- removed R54, R55, R56, R57: 2.2K, symbol R-RESCUE-museV2
- removed U10: PCM1863, symbol PCM1863
- removed U7: PCM9211, symbol PCM9211
- removed X1: 24.576 MHz, symbol CRYSTAL
- renumbered C47 to C35, P2 to P1, R49 to R1, U8 to U1, U11 to U2
Connections:
- net Audio_Filter/ANALOG_OUT+ is gone; now on net Audio_Filter/ANALOG_OUT+: U2.25 (IOUT_L+)
- net Audio_Filter/ANALOG_OUT- is gone; now on net Audio_Filter/ANALOG_OUT-: U2.26 (IOUT_L-)
- net Audio_Filter/ANALOG_OUT+: no longer U2.17 (IOUT_R+)
- net Audio_Filter/ANALOG_OUT-: no longer U2.18 (IOUT_R-)
- new net Audio_Filter/ANALOG_OUT+: U2.17 (IOUT_R+)
- new net Audio_Filter/ANALOG_OUT-: U2.18 (IOUT_R-)
- no-connect marks 45 -> 30
Other:
- note removed: "ADC unused\nAnalog VCC\nGrounded"
- note removed: "Digital Front-End (DFE)"
- note removed: "From ADC\n(Analog In)"
- note removed: "From Edison\n(Bluetooth/\nAnalog input)"
- note removed: "From S/PDIF\n(Digital In)"
- note removed: "From \nMCU(Control)"
- note removed: "I2C Addr 0x80/0x81"
- note removed: "PCM1863 ADC"
- note removed: "Pulled LOW for\nI2C mode"
- note removed: "Pulled LOW for\nI2C mode Addr 0x94"
- note removed: "To DAC\n(Bluetooth/\nDigital/Analog)"
- note removed: "To Edison\n(Digital/Analog\ninput)"
- note removed: "To S/PDIF\n(Digital Out)"
- moved on the sheet: C1, C10, C11, C12, C13, C14, C15, C16, C17, C18, C19, C2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

Commit message: Finished converting to global labels
Parts:
- removed C1, C10, C11, C12, C14, C16, C17, C19, C2, C21, C24, C26, C28, C3, C30, C31, C32, C4, C5, C6, C7, C8, C9: 0.1uF, symbol C-RESCUE-museV2
- removed C13, C15, C18, C20, C22, C23, C25, C27: 10uF, symbol C-RESCUE-museV2
- removed C29: 1uF, symbol C-RESCUE-museV2
- removed C33, C34: 1000uF, symbol C-RESCUE-museV2
- removed C35: 47uF, symbol C-RESCUE-museV2
- removed P1: CONN_01X06, symbol CONN_01X06
- removed R1: 10K, symbol R-RESCUE-museV2
- removed U1: EdisonConnector, symbol EdisonConnector
- removed U2: PCM1796, symbol PCM1796
Connections:
- no-connect marks 30 -> 0
Other:
- note removed: "ADC"
- note removed: "DAC"
- note removed: "DAC Output Filter"
- note removed: "Decoupling"
- note removed: "Digital Front-End"
- note removed: "Edison UART \nInterface"
- note removed: "Intel Edison Connection"
- note removed: "LED Light Connections"
- note removed: "PCM1796 DAC"
- note removed: "PSU Surge Supress"
- note removed: "Pulled HIGH for\nI2C mode"
- note removed: "S/PDIF (I/0)"
- note removed: "To DFE/\n ADC/\n DAC"
- note removed: "To DFE\n(IADC/\n DAC/\n SPDIF)"
- note removed: "To LED\nPWM\ngenerator"
