File: Hardware/POWER.sch (KiCad schematic (older format))
At the start: 16 parts

Commit message: Currently adding level shifters
Parts:
- D? (x2): symbol LED -> LED-RESCUE-museV2
- R? (x2): symbol R -> R-RESCUE-museV2
- U?: symbol LP38692 -> LP38692-RESCUE-museV2
Connections:
- wire segments 119 -> 85
Changed lines of the file:
@@
 LIBS:microchip_pic18mcu
 LIBS:microchip
+LIBS:microchip1
 LIBS:microcontrollers
 LIBS:motorola
@@
 LIBS:sensors
 LIBS:siliconi
+LIBS:special
 LIBS:stm8
 LIBS:stm32
@@
 Text Label 2400 5600 0    60   ~ 0
 EDISON_RST_OUT(1.8)
-Text Label 2450 4150 0    60   ~ 0
+Text Label 3250 4150 2    60   ~ 0
 EDISON_PWR_BTN
 Text Notes 2050 3850 0    60   ~ 0
@@
 $EndComp
 Wire Wire Line
-	3800 4050 3800 4250
-Wire Wire Line
-	3800 4750 3800 4850
+	3800 4050 3800 4350
+Wire Wire Line
+	3800 4650 3800 4850
 Wire Wire Line
 	3800 5250 3800 5350
@@
 Connection ~ 3400 5600
 Wire Wire Line
-	3400 4050 3400 4250
-Wire Wire Line
-	3400 5600 3400 4750
-Wire Wire Line
-	2400 5600 3400 5600
-Wire Wire Line
-	3400 5600 3500 5600
+	3400 4050 3400 4350
+Wire Wire Line
+	3400 4650 3400 5600
+Wire Wire Line
+	2400 5600 3500 5600
 Wire Wire Line
 	2150 5900 2150 5450
 Wire Wire Line
-	2150 4200 2150 4050
+	2150 4050 2150 4300
 Connection ~ 2150 4750
 Wire Wire Line
-	2150 4700 2150 4750
-Wire Wire Line
-	2150 4750 2150 4850
+	2150 4600 2150 4850
 $Comp
 L R-RESCUE-museV2 R?
@@
 $EndComp
 Wire Wire Line
-	2150 4750 2350 4750
+	2350 4750 2150 4750
 $Comp
 L +3.3VSB #PWR?
@@
 $EndComp
 Wire Wire Line
-	2350 4750 2350 4700
+	2350 4600 2350 4750
 Wire Wire Line
 	2350 4150 3250 4150
 Wire Wire Line
-	2350 4200 2350 4150
+	2350 4150 2350 4300
 $Comp
 L +3.3VSB #PWR?
@@
 $EndComp
 $Comp
-L LP38692 U?
+L LP38692-RESCUE-museV2 U?
 U 1 1 57EB0792
 P 5450 4150
@@
 5VSB->3.3VSB LDO
 Wire Wire Line
-	5050 4050 5050 4250
-Wire Wire Line
-	5050 4250 5050 4450
-Wire Wire Line
-	5050 4450 5050 4600
+	5050 4050 5050 4650
 Wire Wire Line
 	5050 4450 5150 4450
@@
 Connection ~ 5050 4250
 Wire Wire Line
-	5700 5150 5700 5250
-Wire Wire Line
-	5700 5250 5700 5350
-Wire Wire Line
-	6350 4050 6350 4250
-Wire Wire Line
-	6350 4250 6350 4600
+	5700 5150 5700 5350
+Wire Wire Line
+	6350 4050 6350 4650
 Connection ~ 5050 4450
 Wire Wire Line
-	5050 5000 5050 5250
-Wire Wire Line
-	5050 5250 5700 5250
-Wire Wire Line
-	5700 5250 6350 5250
+	5050 4950 5050 5250
+Wire Wire Line
+	6350 5250 5050 5250
 Connection ~ 5700 5250
 Wire Wire Line
-	6350 5250 6350 5000
+	6350 4950 6350 5250
 Wire Wire Line
 	6250 4250 6350 4250
@@
 	4500 2400 4400 2400
 Wire Wire Line
-	4400 1900 4400 2400
-Wire Wire Line
-	4400 2400 4400 2500
-Wire Wire Line
-	4400 2500 4400 2600
-Wire Wire Line
-	4400 2600 4400 2700
-Wire Wire Line
-	4400 2700 4400 2800
+	4400 1900 4400 2800
 Wire Wire Line
 	4400 2500 4500 2500
@@
 Connection ~ 4400 2700
 Wire Wire Line
-	4150 1900 4150 3000
-Wire Wire Line
-	4150 3000 4150 3100
+	4150 1900 4150 3100
 Wire Wire Line
 	4150 3000 4500 3000
@@
 	5200 2400 5300 2400
 Wire Wire Line
-	5300 2400 5300 2500
-Wire Wire Line
-	5300 2500 5300 2600
-Wire Wire Line
-	5300 2600 5300 2700
-Wire Wire Line
-	5300 2700 5300 2800
-Wire Wire Line
-	5300 2800 5300 2900
-Wire Wire Line
-	5300 2900 5300 3000
-Wire Wire Line
-	5300 3000 5300 3100
-Wire Wire Line
-	5300 3100 5300 3250
+	5300 2400 5300 3250
 Wire Wire Line
 	5200 2500 5300 2500
@@
 	5200 2300 5900 2300
 Wire Wire Line
-	2500 1900 2500 2000
-Wire Wire Line
-	2500 2000 2500 2100
-Wire Wire Line
-	2500 2100 2500 2200
-Wire Wire Line
-	2500 2200 2500 2300
+	2500 1900 2500 2300
 Wire Wire Line
 	2500 2300 2600 2300
@@
 	2600 2400 2350 2400
 Wire Wire Line
-	2350 1900 2350 2400
-Wire Wire Line
-	2350 2400 2350 2500
-Wire Wire Line
-	2350 2500 2350 2600
-Wire Wire Line
-	2350 2600 2350 2700
-Wire Wire Line
-	2350 2700 2350 2800
+	2350 1900 2350 2800
 Wire Wire Line
 	2350 2500 2600 2500
@@
 	2200 2900 2600 2900
 Wire Wire Line
-	2050 1900 2050 3000
-Wire Wire Line
-	2050 3000 2050 3100
+	2050 1900 2050 3100
 Wire Wire Line
 	2050 3000 2600 3000
@@
 	3300 2400 3400 2400
 Wire Wire Line
-	3400 2400 3400 2500
-Wire Wire Line
-	3400 2500 3400 2600
-Wire Wire Line
-	3400 2600 3400 2700
-Wire Wire Line
-	3400 2700 3400 2800
-Wire Wire Line
-	3400 2800 3400 2900
-Wire Wire Line
-	3400 2900 3400 3000
-Wire Wire Line
-	3400 3000 3400 3100
-Wire Wire Line
-	3400 3100 3400 3250
+	3400 2400 3400 3250
 Wire Wire Line
 	3300 2500 3400 2500
@@
 	2200 2900 2200 1900
 $Comp
-L R R?
+L R-RESCUE-museV2 R?
 U 1 1 57EBFC46
 P 7100 3000
@@
 $EndComp
 $Comp
-L R R?
+L R-RESCUE-museV2 R?
 U 1 1 57EBFCB8
 P 7500 3000
@@
 $EndComp
 $Comp
-L LED D?
+L LED-RESCUE-museV2 D?
 U 1 1 57EBFCF6
 P 7100 2550
@@
 $EndComp
 $Comp
-L LED D?
+L LED-RESCUE-museV2 D?
 U 1 1 57EBFDD5
 P 7500 2550
@@
 $EndComp
 $Comp
-L GND #PWR?
+L GND-RESCUE-museV2 #PWR?
 U 1 1 57EBFE13
 P 7100 3200
@@
 $EndComp
 $Comp
-L GND #PWR?
+L GND-RESCUE-museV2 #PWR?
 U 1 1 57EBFE55
 P 7500 3200

Commit message: In progress changing to global labels
Changed lines of the file:
@@
 LIBS:microchip_pic18mcu
 LIBS:microchip
-LIBS:microchip1
 LIBS:microcontrollers
 LIBS:motorola
@@
 LIBS:sensors
 LIBS:siliconi
-LIBS:special
 LIBS:stm8
 LIBS:stm32
@@
 $Descr A4 11693 8268
 encoding utf-8
-Sheet 7 8
+Sheet 7 9
 Title ""
 Date ""
@@
 	5050 4950 5050 5250
 Wire Wire Line
-	6350 5250 5050 5250
+	5050 5250 6350 5250
 Connection ~ 5700 5250
 Wire Wire Line
-	6350 4950 6350 5250
+	6350 5250 6350 4950
 Wire Wire Line
 	6250 4250 6350 4250

Commit message: Changing to global labels/pages in progress
Parts:
- added P? (x2): 3.5mm_Audio, symbol CONN_01X03
- added P? (x2): RCA_Stero_Jack, symbol RCA_Stero_Jack
- added U?: PLT133/T10W, symbol PLT133/T10W
- added U?: PLR135/T10, symbol PLR135/10
- added U? (x4): POM-3535L-3-R, symbol POM-3535L-3-R
- gave numbers to parts that had none: 16
Connections:
- net labels added: 3.5_IN_L, 3.5_IN_R, ANALOG_OUT_R, MIC_1, MIC_2, MIC_3, MIC_4, RCA_IN_L, RCA_IN_R, SPDIF_IN, SPDIF_OUT
- net labels removed: AUX_PS_2_OK, EDISON_RST_OUT
- wire segments 85 -> 131
Other:
- note added: "Analog Audio Connections"
- note added: "Digital Audio (S/PDIF) Connections"
- note added: "Microphones"
- note added: "Optical In"
- note added: "Optical Output"
- note removed: "Power Signals"
- moved on the sheet: C65, C66, D3, D4, D5, J1, J2, Q14, R120, R121, R122, R123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

Commit message: Finished converting to global labels
Parts:
- added C? (x2): 0.1uF, symbol C-RESCUE-museV2
- added C? (x2): 1000uF, symbol C-RESCUE-museV2
Connections:
- wire segments 131 -> 184
Other:
- note added: "Decoupling Capacitors"
- note added: "PSU Surge Supression\nCapacitors"
- moved on the sheet: P?

Commit message: Made design review fixes, added breakouts
Parts:
- removed C? (x2): 1000uF, symbol C-RESCUE-museV2
- gave numbers to parts that had none: 12
- renumbered C65 to C11, C66 to C12, D5 to D3, D3 to D4, D4 to D5, Q14 to Q2, R120 to R10, R121 to R11, R124 to R6, R125 to R7, R122 to R8, R123 to R9, U14 to U2
Connections:
- net labels removed: -12V, -5V
- wire segments 184 -> 131
- no-connect marks 8 -> 10
Other:
- note removed: "PSU Surge Supression\nCapacitors"

Commit message: Annotated schematic
Parts:
- renumbered C15 to C13, C16 to C14, D4 to D3, D5 to D4, D3 to D5, P3 to P2, P2 to P3, R8 to R10, R9 to R11, R10 to R6, R11 to R7, R6 to R8, R7 to R9, U5 to U4, U6 to U5, U4 to U6

Commit message: Pushing most updated version
Parts:
- removed P1, P2: RCA_Stero_Jack, symbol RCA_Stero_Jack
- removed U2: LP38692, symbol LP38692-RESCUE-museV2
- added P1: RCA_STEREO_JACK, symbol CONN_01X06
- added U2: LP38692, symbol LP38692SD
Connections:
- net +3.3VSB: now also U2.4 (OUT), U2.5 (SNS)
- net +5VSB: now also U2.1 (IN), U2.3 (EN), U2.6 (IN)
- net ANALOG_OUT_R: now also P1.3 (P3); no longer P4.2 (P2)
- net GND: now also P1.5 (P5), P1.6 (P6), U2.2 (GND)
- net RCA_IN_L: now also P1.2 (P2)
- net RCA_IN_R: now also P1.1 (P1)
- new net ANALOG_OUT_L: P1.4 (P4), P4.2 (P2)
- no-connect marks 10 -> 9
Other:
- moved on the sheet: C12, P3, P4
