File: Hardware/DAC.sch (KiCad schematic (older format))
At the start: 10 parts

Commit message: Updated I2C pullup resistors and labels
Connections:
- net labels added: I2S_DAC_BCK(3.3), I2S_DAC_DIN(3.3), I2S_DAC_LRCK(3.3), I2S_SCK(3.3)
- net labels removed: I2S_DAC_BCK, I2S_DAC_DIN, I2S_DAC_LRCK, I2S_SCK
- wire segments 81 -> 89
Other:
- moved on the sheet: C?
Changed lines of the file:
@@
 Comment4 ""
 $EndDescr
-Text Notes 3650 5350 0    60   ~ 0
+Text Notes 2950 5350 0    60   ~ 0
 Pulled HIGH for\nI2C mode
 $Comp
@@
 F4 "ANALOG_OUT" I R 7950 4700 60
 $EndSheet
-Text Label 3750 4550 0    60   ~ 0
-I2S_SCK
-Text Label 3750 4900 0    60   ~ 0
-I2C_SCL(3.3)
-Text Label 3750 5000 0    60   ~ 0
-I2C_SDA(3.3)
-Text Label 3750 4400 0    60   ~ 0
-I2S_DAC_BCK
-Text Label 3750 4300 0    60   ~ 0
-I2S_DAC_DIN
-Text Label 3750 4200 0    60   ~ 0
-I2S_DAC_LRCK
-Text Label 3750 3900 0    60   ~ 0
-DAC_RST
 $Comp
 L PCM1796 U?
@@
 L GND-RESCUE-museV2 #PWR?
 U 1 1 57F8A564
-P 6100 5600
-F 0 "#PWR?" H 6100 5600 30  0001 C CNN
-F 1 "GND" H 6100 5530 30  0001 C CNN
-F 2 "" H 6100 5600 60  0000 C CNN
-F 3 "" H 6100 5600 60  0000 C CNN
-	1    6100 5600
+P 6100 5450
+F 0 "#PWR?" H 6100 5450 30  0001 C CNN
+F 1 "GND" H 6100 5380 30  0001 C CNN
+F 2 "" H 6100 5450 60  0000 C CNN
+F 3 "" H 6100 5450 60  0000 C CNN
+	1    6100 5450
 	1    0    0    -1
 $EndComp
@@
 L GND-RESCUE-museV2 #PWR?
 U 1 1 57F8A571
-P 5800 5600
-F 0 "#PWR?" H 5800 5600 30  0001 C CNN
-F 1 "GND" H 5800 5530 30  0001 C CNN
-F 2 "" H 5800 5600 60  0000 C CNN
-F 3 "" H 5800 5600 60  0000 C CNN
-	1    5800 5600
+P 5800 5450
+F 0 "#PWR?" H 5800 5450 30  0001 C CNN
+F 1 "GND" H 5800 5380 30  0001 C CNN
+F 2 "" H 5800 5450 60  0000 C CNN
+F 3 "" H 5800 5450 60  0000 C CNN
+	1    5800 5450
 	1    0    0    -1
 $EndComp
@@
 L C-RESCUE-museV2 C?
 U 1 1 57F8A577
-P 3500 3850
-F 0 "C?" H 3500 3950 40  0000 L CNN
-F 1 "47uF" H 3506 3765 40  0000 L CNN
-F 2 "" H 3538 3700 30  0000 C CNN
-F 3 "" H 3500 3850 60  0000 C CNN
-	1    3500 3850
-	1    0    0    -1
-$EndComp
-Text Notes 3400 2350 0    60   ~ 0
+P 2800 3850
+F 0 "C?" H 2800 3950 40  0000 L CNN
+F 1 "47uF" H 2806 3765 40  0000 L CNN
+F 2 "" H 2838 3700 30  0000 C CNN
+F 3 "" H 2800 3850 60  0000 C CNN
+	1    2800 3850
+	1    0    0    -1
+$EndComp
+Text Notes 2950 2350 0    60   ~ 12
 PCM1796 DAC
 $Comp
 L +3.3VSB #PWR?
 U 1 1 57F8A57F
-P 4300 2600
-F 0 "#PWR?" H 4300 2560 30  0001 C CNN
-F 1 "+3.3VSB" H 4300 2710 30  0000 C CNN
-F 2 "" H 4300 2600 60  0000 C CNN
-F 3 "" H 4300 2600 60  0000 C CNN
-	1    4300 2600
+P 4300 3300
+F 0 "#PWR?" H 4300 3260 30  0001 C CNN
+F 1 "+3.3VSB" H 4300 3410 30  0000 C CNN
+F 2 "" H 4300 3300 60  0000 C CNN
+F 3 "" H 4300 3300 60  0000 C CNN
+	1    4300 3300
 	1    0    0    -1
 $EndComp
@@
 L +5VSB #PWR?
 U 1 1 57F8A585
-P 3500 2600
-F 0 "#PWR?" H 3500 2690 20  0001 C CNN
-F 1 "+5VSB" H 3500 2690 30  0000 C CNN
-F 2 "" H 3500 2600 60  0000 C CNN
-F 3 "" H 3500 2600 60  0000 C CNN
-	1    3500 2600
+P 2800 3300
+F 0 "#PWR?" H 2800 3390 20  0001 C CNN
+F 1 "+5VSB" H 2800 3390 30  0000 C CNN
+F 2 "" H 2800 3300 60  0000 C CNN
+F 3 "" H 2800 3300 60  0000 C CNN
+	1    2800 3300
 	1    0    0    -1
 $EndComp
@@
 L +5VSB #PWR?
 U 1 1 57F8A58B
-P 5800 2600
-F 0 "#PWR?" H 5800 2690 20  0001 C CNN
-F 1 "+5VSB" H 5800 2690 30  0000 C CNN
-F 2 "" H 5800 2600 60  0000 C CNN
-F 3 "" H 5800 2600 60  0000 C CNN
-	1    5800 2600
+P 5800 3300
+F 0 "#PWR?" H 5800 3390 20  0001 C CNN
+F 1 "+5VSB" H 5800 3390 30  0000 C CNN
+F 2 "" H 5800 3300 60  0000 C CNN
+F 3 "" H 5800 3300 60  0000 C CNN
+	1    5800 3300
 	1    0    0    -1
 $EndComp
@@
 L +3.3VSB #PWR?
 U 1 1 57F8A593
-P 3500 4500
-F 0 "#PWR?" H 3500 4460 30  0001 C CNN
-F 1 "+3.3VSB" H 3500 4610 30  0000 C CNN
-F 2 "" H 3500 4500 60  0000 C CNN
-F 3 "" H 3500 4500 60  0000 C CNN
-	1    3500 4500
-	1    0    0    -1
-$EndComp
-Wire Wire Line
-	4300 2600 4300 3450
+P 2800 4500
+F 0 "#PWR?" H 2800 4460 30  0001 C CNN
+F 1 "+3.3VSB" H 2800 4610 30  0000 C CNN
+F 2 "" H 2800 4500 60  0000 C CNN
+F 3 "" H 2800 4500 60  0000 C CNN
+	1    2800 4500
+	1    0    0    -1
+$EndComp
+Text GLabel 4100 3900 0    60   Input ~ 0
+DAC_RST
+Text GLabel 4100 4100 0    60   Input ~ 0
+I2S_DAC_LRCK(3.3)
+Text GLabel 4100 4250 0    60   Input ~ 0
+I2S_DAC_DIN(3.3)
+Text GLabel 4100 4400 0    60   Input ~ 0
+I2S_DAC_BCK(3.3)
+Text GLabel 4100 4550 0    60   Input ~ 0
+I2S_SCK(3.3)
+Text GLabel 4100 4900 0    60   Input ~ 0
+I2C_SCL(3.3)
+Text GLabel 4100 5050 0    60   Input ~ 0
+I2C_SDA(3.3)
+Wire Wire Line
+	4300 3300 4300 3450
 Wire Wire Line
 	4300 3450 4400 3450
 Wire Wire Line
-	3700 3750 4400 3750
-Wire Wire Line
-	3500 2600 3500 3550
-Wire Wire Line
-	3500 3550 3500 3700
-Connection ~ 3500 3550
-Wire Wire Line
-	3700 3650 3700 3750
-Wire Wire Line
-	3700 3750 3700 4100
-Wire Wire Line
-	4400 3650 3700 3650
-Connection ~ 3700 3750
-Wire Wire Line
-	3700 4100 3500 4100
-Wire Wire Line
-	3500 4100 3500 4000
+	2800 3300 2800 3550
+Wire Wire Line
+	2800 3550 2800 3700
+Connection ~ 2800 3550
+Wire Wire Line
+	3000 3650 3000 4100
+Wire Wire Line
+	3000 3650 4300 3650
+Wire Wire Line
+	4300 3650 4400 3650
+Wire Wire Line
+	3000 4100 2800 4100
+Wire Wire Line
+	2800 4100 2800 4000
 Wire Wire Line
 	5700 4050 6500 4050
 Wire Wire Line
-	3750 3900 4400 3900
-Wire Wire Line
-	4400 4200 3750 4200
-Wire Wire Line
-	4400 4300 3750 4300
-Wire Wire Line
-	4400 4400 3750 4400
-Wire Wire Line
-	4400 4550 3750 4550
-Wire Wire Line
-	4400 5000 3750 5000
-Wire Wire Line
-	4400 4900 3750 4900
+	4100 3900 4400 3900
+Wire Wire Line
+	4400 4200 4300 4200
+Wire Wire Line
+	4200 4300 4400 4300
+Wire Wire Line
+	4400 4400 4100 4400
+Wire Wire Line
+	4400 4550 4100 4550
 Wire Wire Line
 	5800 4750 5800 4850
@@
 	5800 5050 5800 5150
 Wire Wire Line
-	5800 5150 5800 5600
+	5800 5150 5800 5450
 Wire Wire Line
 	5800 5150 5700 5150
@@
 	6100 4550 6100 5000
 Wire Wire Line
-	6100 5300 6100 5600
+	6100 5300 6100 5450
 Wire Wire Line
 	5700 4150 6500 4150
@@
 	5800 3550 5700 3550
 Wire Wire Line
-	5800 2600 5800 3450
+	5800 3300 5800 3450
 Wire Wire Line
 	5800 3450 5800 3550
@@
 Connection ~ 5800 4850
 Wire Wire Line
-	3500 3550 4400 3550
+	2800 3550 4400 3550
 Wire Wire Line
 	6250 4350 6250 4750
@@
 Connection ~ 8150 3250
 Wire Wire Line
-	3500 4500 3500 4700
-Wire Wire Line
-	3500 4700 3500 4800
-Wire Wire Line
-	3500 4800 3500 5150
-Wire Wire Line
-	3500 5150 4400 5150
-Wire Wire Line
-	4400 4800 3500 4800
-Connection ~ 3500 4800
-Wire Wire Line
-	4400 4700 3500 4700
-Connection ~ 3500 4700
+	2800 4500 2800 4700
+Wire Wire Line
+	2800 4700 2800 5150
+Connection ~ 2800 4700
+Wire Wire Line
+	4200 4300 4200 4250
+Wire Wire Line
+	4200 4250 4100 4250
+Wire Wire Line
+	4300 4200 4300 4100
+Wire Wire Line
+	4300 4100 4100 4100
+Wire Wire Line
+	4400 3750 4300 3750
+Wire Wire Line
+	4300 3750 4300 3650
+Connection ~ 4300 3650
+Wire Wire Line
+	4100 4900 4400 4900
+Wire Wire Line
+	4100 5050 4200 5050
+Wire Wire Line
+	4200 5050 4200 5000
+Wire Wire Line
+	4200 5000 4400 5000
+Wire Wire Line
+	4400 4800 4300 4800
+Wire Wire Line
+	4300 4800 4300 4700
+Connection ~ 4300 4700
+Wire Wire Line
+	2800 5150 4400 5150
+Wire Wire Line
+	2800 4700 4300 4700
+Wire Wire Line
+	4300 4700 4400 4700
 $EndSCHEMATC

Commit message: Made design review fixes, added breakouts
Parts:
- gave numbers to parts that had none: 10
Changed lines of the file:
@@
 LIBS:microchip_pic18mcu
 LIBS:microchip
-LIBS:microchip1
 LIBS:microcontrollers
 LIBS:motorola
@@
 LIBS:sensors
 LIBS:siliconi
-LIBS:special
 LIBS:stm8
 LIBS:stm32
@@
 Pulled HIGH for\nI2C mode
 $Comp
-L GND-RESCUE-museV2 #PWR?
+L GND-RESCUE-museV2 #PWR88
 U 1 1 57F8A4EE
 P 8150 3350
-F 0 "#PWR?" H 8150 3350 30  0001 C CNN
+F 0 "#PWR88" H 8150 3350 30  0001 C CNN
 F 1 "GND" H 8150 3280 30  0001 C CNN
 F 2 "" H 8150 3350 60  0000 C CNN
@@
 $EndComp
 $Comp
-L C-RESCUE-museV2 C?
+L C-RESCUE-museV2 C51
 U 1 1 57F8A4F4
 P 8300 2950
-F 0 "C?" H 8300 3050 40  0000 L CNN
+F 0 "C51" H 8300 3050 40  0000 L CNN
 F 1 "0.1uF" H 8306 2865 40  0000 L CNN
 F 2 "" H 8338 2800 30  0000 C CNN
@@
 $EndComp
 $Comp
-L C-RESCUE-museV2 C?
+L C-RESCUE-museV2 C50
 U 1 1 57F8A4FB
 P 8000 2950
-F 0 "C?" H 8000 3050 40  0000 L CNN
+F 0 "C50" H 8000 3050 40  0000 L CNN
 F 1 "10uF" H 8006 2865 40  0000 L CNN
 F 2 "" H 8038 2800 30  0000 C CNN
@@
 $EndComp
 $Comp
-L +3.3V-RESCUE-museV2 #PWR?
+L +3.3V-RESCUE-museV2 #PWR87
 U 1 1 57F8A502
 P 8150 2600
-F 0 "#PWR?" H 8150 2560 30  0001 C CNN
+F 0 "#PWR87" H 8150 2560 30  0001 C CNN
 F 1 "+3.3V" H 8150 2710 30  0000 C CNN
 F 2 "" H 8150 2600 60  0000 C CNN
@@
 $EndComp
 $Comp
-L +5V #PWR?
+L +5V #PWR85
 U 1 1 57F8A508
 P 7100 2600
-F 0 "#PWR?" H 7100 2690 20  0001 C CNN
+F 0 "#PWR85" H 7100 2690 20  0001 C CNN
 F 1 "+5V" H 7100 2690 30  0000 C CNN
 F 2 "" H 7100 2600 60  0000 C CNN
@@
 Decoupling Capacitors
 $Comp
-L GND-RESCUE-museV2 #PWR?
+L GND-RESCUE-museV2 #PWR86
 U 1 1 57F8A50F
 P 7100 3350
-F 0 "#PWR?" H 7100 3350 30  0001 C CNN
+F 0 "#PWR86" H 7100 3350 30  0001 C CNN
 F 1 "GND" H 7100 3280 30  0001 C CNN
 F 2 "" H 7100 3350 60  0000 C CNN
@@
 $EndComp
 $Comp
-L C-RESCUE-museV2 C?
+L C-RESCUE-museV2 C49
 U 1 1 57F8A515
 P 7700 2950
-F 0 "C?" H 7700 3050 40  0000 L CNN
+F 0 "C49" H 7700 3050 40  0000 L CNN
 F 1 "10uF" H 7706 2865 40  0000 L CNN
 F 2 "" H 7738 2800 30  0000 C CNN
@@
 $EndComp
 $Comp
-L C-RESCUE-museV2 C?
+L C-RESCUE-museV2 C48
 U 1 1 57F8A51C
 P 7400 2950
-F 0 "C?" H 7400 3050 40  0000 L CNN
+F 0 "C48" H 7400 3050 40  0000 L CNN
 F 1 "0.1uF" H 7406 2865 40  0000 L CNN
 F 2 "" H 7438 2800 30  0000 C CNN
@@
 $EndComp
 $Comp
-L C-RESCUE-museV2 C?
+L C-RESCUE-museV2 C47
 U 1 1 57F8A523
 P 7100 2950
-F 0 "C?" H 7100 3050 40  0000 L CNN
+F 0 "C47" H 7100 3050 40  0000 L CNN
 F 1 "10uF" H 7106 2865 40  0000 L CNN
 F 2 "" H 7138 2800 30  0000 C CNN
@@
 $EndComp
 $Comp
-L C-RESCUE-museV2 C?
+L C-RESCUE-museV2 C46
 U 1 1 57F8A52A
 P 6800 2950
-F 0 "C?" H 6800 3050 40  0000 L CNN
+F 0 "C46" H 6800 3050 40  0000 L CNN
 F 1 "0.1uF" H 6806 2865 40  0000 L CNN
 F 2 "" H 6838 2800 30  0000 C CNN
@@
 $EndComp
 $Comp
-L C-RESCUE-museV2 C?
+L C-RESCUE-museV2 C45
 U 1 1 57F8A531
 P 6500 2950
-F 0 "C?" H 6500 3050 40  0000 L CNN
+F 0 "C45" H 6500 3050 40  0000 L CNN
 F 1 "10uF" H 6506 2865 40  0000 L CNN
 F 2 "" H 6538 2800 30  0000 C CNN
@@
 	1    0    0    -1
 $EndComp
-Text Label 8750 4700 2    60   ~ 0
-ANALOG_OUT_R
-Text Label 8750 4100 2    60   ~ 0
-ANALOG_OUT_L
 $Sheet
 S 6500 3950 1450 300
@@
 $EndSheet
 $Comp
-L PCM1796 U?
+L PCM1796 U11
 U 1 1 57F8A55D
 P 4600 3400
-F 0 "U?" H 4700 3450 60  0000 C CNN
+F 0 "U11" H 4700 3450 60  0000 C CNN
 F 1 "PCM1796" H 5300 1500 60  0000 C CNN
 F 2 "" H 4600 3400 60  0000 C CNN
@@
 $EndComp
 $Comp
-L GND-RESCUE-museV2 #PWR?
+L GND-RESCUE-museV2 #PWR84
 U 1 1 57F8A564
 P 6100 5450
-F 0 "#PWR?" H 6100 5450 30  0001 C CNN
+F 0 "#PWR84" H 6100 5450 30  0001 C CNN
 F 1 "GND" H 6100 5380 30  0001 C CNN
 F 2 "" H 6100 5450 60  0000 C CNN
@@
 $EndComp
 $Comp
-L R-RESCUE-museV2 R?
+L R-RESCUE-museV2 R25
 U 1 1 57F8A56A
 P 6100 5150
-F 0 "R?" V 6180 5150 40  0000 C CNN
+F 0 "R25" V 6180 5150 40  0000 C CNN
 F 1 "10K" V 6107 5151 40  0000 C CNN
 F 2 "" V 6030 5150 30  0000 C CNN
@@
 $EndComp
 $Comp
-L GND-RESCUE-museV2 #PWR?
+L GND-RESCUE-museV2 #PWR83
 U 1 1 57F8A571
 P 5800 5450
-F 0 "#PWR?" H 5800 5450 30  0001 C CNN
+F 0 "#PWR83" H 5800 5450 30  0001 C CNN
 F 1 "GND" H 5800 5380 30  0001 C CNN
 F 2 "" H 5800 5450 60  0000 C CNN
@@
 $EndComp
 $Comp
-L C-RESCUE-museV2 C?
+L C-RESCUE-museV2 C44
 U 1 1 57F8A577
 P 2800 3850
-F 0 "C?" H 2800 3950 40  0000 L CNN
+F 0 "C44" H 2800 3950 40  0000 L CNN
 F 1 "47uF" H 2806 3765 40  0000 L CNN
 F 2 "" H 2838 3700 30  0000 C CNN
@@
 PCM1796 DAC
 $Comp
-L +3.3VSB #PWR?
+L +3.3VSB #PWR81
 U 1 1 57F8A57F
 P 4300 3300
-F 0 "#PWR?" H 4300 3260 30  0001 C CNN
+F 0 "#PWR81" H 4300 3260 30  0001 C CNN
 F 1 "+3.3VSB" H 4300 3410 30  0000 C CNN
 F 2 "" H 4300 3300 60  0000 C CNN
@@
 $EndComp
 $Comp
-L +5VSB #PWR?
+L +5VSB #PWR79
 U 1 1 57F8A585
 P 2800 3300
-F 0 "#PWR?" H 2800 3390 20  0001 C CNN
+F 0 "#PWR79" H 2800 3390 20  0001 C CNN
 F 1 "+5VSB" H 2800 3390 30  0000 C CNN
 F 2 "" H 2800 3300 60  0000 C CNN
@@
 $EndComp
 $Comp
-L +5VSB #PWR?
+L +5VSB #PWR82
 U 1 1 57F8A58B
 P 5800 3300
-F 0 "#PWR?" H 5800 3390 20  0001 C CNN
+F 0 "#PWR82" H 5800 3390 20  0001 C CNN
 F 1 "+5VSB" H 5800 3390 30  0000 C CNN
 F 2 "" H 5800 3300 60  0000 C CNN
@@
 NoConn ~ 5700 3850
 $Comp
-L +3.3VSB #PWR?
+L +3.3VSB #PWR80
 U 1 1 57F8A593
 P 2800 4500
-F 0 "#PWR?" H 2800 4460 30  0001 C CNN
+F 0 "#PWR80" H 2800 4460 30  0001 C CNN
 F 1 "+3.3VSB" H 2800 4610 30  0000 C CNN
 F 2 "" H 2800 4500 60  0000 C CNN
@@
 	6350 4650 6350 4250
 Wire Wire Line
-	7950 4700 8750 4700
-Wire Wire Line
-	7950 4100 8750 4100
+	7950 4700 8250 4700
+Wire Wire Line
+	7950 4100 8250 4100
 Wire Wire Line
 	7100 2600 7100 2650
@@
 Wire Wire Line
 	4300 4700 4400 4700
+Text GLabel 8250 4100 2    60   Input ~ 0
+ANALOG_OUT_L
+Text GLabel 8250 4700 2    60   Input ~ 0
+ANALOG_OUT_R
 $EndSCHEMATC

Commit message: Annotated schematic
Parts:
- renumbered C45 to C42, C46 to C43, C47 to C44, C48 to C45, C49 to C46, C50 to C47, C51 to C48, C44 to C49
Connections:
- wire segments 89 -> 70
Changed lines of the file:
@@
 LIBS:microchip_pic18mcu
 LIBS:microchip
+LIBS:microchip1
 LIBS:microcontrollers
 LIBS:motorola
@@
 LIBS:sensors
 LIBS:siliconi
+LIBS:special
 LIBS:stm8
 LIBS:stm32
@@
 Pulled HIGH for\nI2C mode
 $Comp
-L GND-RESCUE-museV2 #PWR88
+L GND-RESCUE-museV2-RESCUE-museV2 #PWR074
 U 1 1 57F8A4EE
 P 8150 3350
-F 0 "#PWR88" H 8150 3350 30  0001 C CNN
+F 0 "#PWR074" H 8150 3350 30  0001 C CNN
 F 1 "GND" H 8150 3280 30  0001 C CNN
 F 2 "" H 8150 3350 60  0000 C CNN
@@
 $EndComp
 $Comp
-L C-RESCUE-museV2 C51
+L C-RESCUE-museV2 C48
 U 1 1 57F8A4F4
 P 8300 2950
-F 0 "C51" H 8300 3050 40  0000 L CNN
+F 0 "C48" H 8300 3050 40  0000 L CNN
 F 1 "0.1uF" H 8306 2865 40  0000 L CNN
 F 2 "" H 8338 2800 30  0000 C CNN
@@
 $EndComp
 $Comp
-L C-RESCUE-museV2 C50
+L C-RESCUE-museV2 C47
 U 1 1 57F8A4FB
 P 8000 2950
-F 0 "C50" H 8000 3050 40  0000 L CNN
+F 0 "C47" H 8000 3050 40  0000 L CNN
 F 1 "10uF" H 8006 2865 40  0000 L CNN
 F 2 "" H 8038 2800 30  0000 C CNN
@@
 $EndComp
 $Comp
-L +3.3V-RESCUE-museV2 #PWR87
+L +3.3V-RESCUE-museV2 #PWR075
 U 1 1 57F8A502
 P 8150 2600
-F 0 "#PWR87" H 8150 2560 30  0001 C CNN
+F 0 "#PWR075" H 8150 2560 30  0001 C CNN
 F 1 "+3.3V" H 8150 2710 30  0000 C CNN
 F 2 "" H 8150 2600 60  0000 C CNN
@@
 $EndComp
 $Comp
-L +5V #PWR85
+L +5V #PWR076
 U 1 1 57F8A508
 P 7100 2600
-F 0 "#PWR85" H 7100 2690 20  0001 C CNN
+F 0 "#PWR076" H 7100 2690 20  0001 C CNN
 F 1 "+5V" H 7100 2690 30  0000 C CNN
 F 2 "" H 7100 2600 60  0000 C CNN
@@
 Decoupling Capacitors
 $Comp
-L GND-RESCUE-museV2 #PWR86
+L GND-RESCUE-museV2-RESCUE-museV2 #PWR077
 U 1 1 57F8A50F
 P 7100 3350
-F 0 "#PWR86" H 7100 3350 30  0001 C CNN
+F 0 "#PWR077" H 7100 3350 30  0001 C CNN
 F 1 "GND" H 7100 3280 30  0001 C CNN
 F 2 "" H 7100 3350 60  0000 C CNN
@@
 $EndComp
 $Comp
-L C-RESCUE-museV2 C49
+L C-RESCUE-museV2 C46
 U 1 1 57F8A515
 P 7700 2950
-F 0 "C49" H 7700 3050 40  0000 L CNN
+F 0 "C46" H 7700 3050 40  0000 L CNN
 F 1 "10uF" H 7706 2865 40  0000 L CNN
 F 2 "" H 7738 2800 30  0000 C CNN
@@
 $EndComp
 $Comp
-L C-RESCUE-museV2 C48
+L C-RESCUE-museV2 C45
 U 1 1 57F8A51C
 P 7400 2950
-F 0 "C48" H 7400 3050 40  0000 L CNN
+F 0 "C45" H 7400 3050 40  0000 L CNN
 F 1 "0.1uF" H 7406 2865 40  0000 L CNN
 F 2 "" H 7438 2800 30  0000 C CNN
@@
 $EndComp
 $Comp
-L C-RESCUE-museV2 C47
+L C-RESCUE-museV2 C44
 U 1 1 57F8A523
 P 7100 2950
-F 0 "C47" H 7100 3050 40  0000 L CNN
+F 0 "C44" H 7100 3050 40  0000 L CNN
 F 1 "10uF" H 7106 2865 40  0000 L CNN
 F 2 "" H 7138 2800 30  0000 C CNN
@@
 $EndComp
 $Comp
-L C-RESCUE-museV2 C46
+L C-RESCUE-museV2 C43
 U 1 1 57F8A52A
 P 6800 2950
-F 0 "C46" H 6800 3050 40  0000 L CNN
+F 0 "C43" H 6800 3050 40  0000 L CNN
 F 1 "0.1uF" H 6806 2865 40  0000 L CNN
 F 2 "" H 6838 2800 30  0000 C CNN
@@
 $EndComp
 $Comp
-L C-RESCUE-museV2 C45
+L C-RESCUE-museV2 C42
 U 1 1 57F8A531
 P 6500 2950
-F 0 "C45" H 6500 3050 40  0000 L CNN
+F 0 "C42" H 6500 3050 40  0000 L CNN
 F 1 "10uF" H 6506 2865 40  0000 L CNN
 F 2 "" H 6538 2800 30  0000 C CNN
@@
 $EndComp
 $Comp
-L GND-RESCUE-museV2 #PWR84
+L GND-RESCUE-museV2-RESCUE-museV2 #PWR078
 U 1 1 57F8A564
 P 6100 5450
-F 0 "#PWR84" H 6100 5450 30  0001 C CNN
+F 0 "#PWR078" H 6100 5450 30  0001 C CNN
 F 1 "GND" H 6100 5380 30  0001 C CNN
 F 2 "" H 6100 5450 60  0000 C CNN
@@
 $EndComp
 $Comp
-L GND-RESCUE-museV2 #PWR83
+L GND-RESCUE-museV2-RESCUE-museV2 #PWR079
 U 1 1 57F8A571
 P 5800 5450
-F 0 "#PWR83" H 5800 5450 30  0001 C CNN
+F 0 "#PWR079" H 5800 5450 30  0001 C CNN
 F 1 "GND" H 5800 5380 30  0001 C CNN
 F 2 "" H 5800 5450 60  0000 C CNN
@@
 $EndComp
 $Comp
-L C-RESCUE-museV2 C44
+L C-RESCUE-museV2 C49
 U 1 1 57F8A577
 P 2800 3850
-F 0 "C44" H 2800 3950 40  0000 L CNN
+F 0 "C49" H 2800 3950 40  0000 L CNN
 F 1 "47uF" H 2806 3765 40  0000 L CNN
 F 2 "" H 2838 3700 30  0000 C CNN
@@
 PCM1796 DAC
 $Comp
-L +3.3VSB #PWR81
+L +3.3VSB #PWR080
 U 1 1 57F8A57F
 P 4300 3300
-F 0 "#PWR81" H 4300 3260 30  0001 C CNN
+F 0 "#PWR080" H 4300 3260 30  0001 C CNN
 F 1 "+3.3VSB" H 4300 3410 30  0000 C CNN
 F 2 "" H 4300 3300 60  0000 C CNN
@@
 $EndComp
 $Comp
-L +5VSB #PWR79
+L +5VSB #PWR081
 U 1 1 57F8A585
 P 2800 3300
-F 0 "#PWR79" H 2800 3390 20  0001 C CNN
+F 0 "#PWR081" H 2800 3390 20  0001 C CNN
 F 1 "+5VSB" H 2800 3390 30  0000 C CNN
 F 2 "" H 2800 3300 60  0000 C CNN
@@
 $EndComp
 $Comp
-L +5VSB #PWR82
+L +5VSB #PWR082
 U 1 1 57F8A58B
 P 5800 3300
-F 0 "#PWR82" H 5800 3390 20  0001 C CNN
+F 0 "#PWR082" H 5800 3390 20  0001 C CNN
 F 1 "+5VSB" H 5800 3390 30  0000 C CNN
 F 2 "" H 5800 3300 60  0000 C CNN
@@
 NoConn ~ 5700 3850
 $Comp
-L +3.3VSB #PWR80
+L +3.3VSB #PWR083
 U 1 1 57F8A593
 P 2800 4500
-F 0 "#PWR80" H 2800 4460 30  0001 C CNN
+F 0 "#PWR083" H 2800 4460 30  0001 C CNN
 F 1 "+3.3VSB" H 2800 4610 30  0000 C CNN
 F 2 "" H 2800 4500 60  0000 C CNN
@@
 	4300 3450 4400 3450
 Wire Wire Line
-	2800 3300 2800 3550
-Wire Wire Line
-	2800 3550 2800 3700
+	2800 3300 2800 3700
 Connection ~ 2800 3550
 Wire Wire Line
 	3000 3650 3000 4100
 Wire Wire Line
-	3000 3650 4300 3650
-Wire Wire Line
-	4300 3650 4400 3650
+	3000 3650 4400 3650
 Wire Wire Line
 	3000 4100 2800 4100
@@
 	4400 4550 4100 4550
 Wire Wire Line
-	5800 4750 5800 4850
-Wire Wire Line
-	5800 4850 5800 4950
-Wire Wire Line
-	5800 4950 5800 5050
-Wire Wire Line
-	5800 5050 5800 5150
-Wire Wire Line
-	5800 5150 5800 5450
+	5800 4750 5800 5450
 Wire Wire Line
 	5800 5150 5700 5150
@@
 	5800 3550 5700 3550
 Wire Wire Line
-	5800 3300 5800 3450
-Wire Wire Line
-	5800 3450 5800 3550
+	5800 3300 5800 3550
 Wire Wire Line
 	5700 3450 5800 3450
@@
 	7950 4100 8250 4100
 Wire Wire Line
-	7100 2600 7100 2650
-Wire Wire Line
-	7100 2650 7100 2800
-Wire Wire Line
-	6500 2650 6800 2650
-Wire Wire Line
-	6800 2650 7100 2650
-Wire Wire Line
-	7100 2650 7400 2650
-Wire Wire Line
-	7400 2650 7700 2650
+	7100 2600 7100 2800
+Wire Wire Line
+	6500 2650 7700 2650
 Wire Wire Line
 	6800 2650 6800 2800
@@
 Connection ~ 7400 2650
 Wire Wire Line
-	6500 3250 6800 3250
-Wire Wire Line
-	6800 3250 7100 3250
-Wire Wire Line
-	7100 3250 7400 3250
-Wire Wire Line
-	7400 3250 7700 3250
+	6500 3250 7700 3250
 Wire Wire Line
 	7400 3100 7400 3250
 Connection ~ 7400 3250
 Wire Wire Line
-	7100 3100 7100 3250
-Wire Wire Line
-	7100 3250 7100 3350
+	7100 3100 7100 3350
 Wire Wire Line
 	6800 3100 6800 3250
@@
 	8000 2650 8000 2800
 Wire Wire Line
-	8000 2650 8150 2650
-Wire Wire Line
-	8150 2650 8300 2650
+	8000 2650 8300 2650
 Wire Wire Line
 	8150 2650 8150 2600
@@
 	8000 3100 8000 3250
 Wire Wire Line
-	8000 3250 8150 3250
-Wire Wire Line
-	8150 3250 8300 3250
+	8000 3250 8300 3250
 Wire Wire Line
 	8150 3250 8150 3350
@@
 Connection ~ 8150 3250
 Wire Wire Line
-	2800 4500 2800 4700
-Wire Wire Line
-	2800 4700 2800 5150
+	2800 4500 2800 5150
 Connection ~ 2800 4700
 Wire Wire Line
@@
 	2800 5150 4400 5150
 Wire Wire Line
-	2800 4700 4300 4700
-Wire Wire Line
-	4300 4700 4400 4700
+	2800 4700 4400 4700
 Text GLabel 8250 4100 2    60   Input ~ 0
 ANALOG_OUT_L
