File: Hardware/DAC.sch (KiCad schematic (older format))
At the start: 10 parts, among them U11 PCM1796

Commit message: Op-Amp placement and wiring
Parts:
- C46: footprint Capacitors_SMD:c_elec_4x5.3 -> Capacitors_SMD:C_0402
Changed lines of the file:
@@
 F 0 "C46" H 7700 3050 40  0000 L CNN
 F 1 "0.1uF" H 7706 2865 40  0000 L CNN
-F 2 "Capacitors_SMD:c_elec_4x5.3" H 7738 2800 30  0001 C CNN
+F 2 "Capacitors_SMD:C_0402" H 7738 2800 30  0001 C CNN
 F 3 "" H 7700 2950 60  0000 C CNN
 	1    7700 2950
