File: Hardware/LEVEL_SHIFTER.sch (KiCad schematic (older format))
At the start: 73 parts, among them U19 GTL2010, U20 GTL2010, U21 GTL2010

Commit message: Fixed schematic errors, added muse-v2-lib
Parts:
- C78, C79, C80: footprint (none) -> Capacitors_SMD:C_0402
- R100, R101, R102, R103, R104, R105, R106, R107, R108, R109, R110, R44, R45, R46, R47, R48, R49, R50, R51, R52, R53, R54, R55, R56, R57, R58, R59, R60, R61, R62, R63, R64, R65, R66, R67, R68, R69, R70, R71, R72, R73, R74, R75, R76, R77, R78, R79, R80, R81, R82, R83, R84, R85, R86, R95, R96, R97, R98, R99: footprint (none) -> Resistors_SMD:R_0402
- R87, R88, R89, R90, R91, R92, R93, R94: footprint (none) -> Resistors_Universal:Resistor_SMD+THTuniversal_0805to1206_RM10_HandSoldering

Commit message: Added proper audio connectors to schematic
Parts:
- U19, U20, U21: footprint (none) -> Housings_SSOP:SSOP-24_5.3x8.2mm_Pitch0.65mm
Changed lines of the file:
@@
 $EndDescr
 $Comp
-L GND-RESCUE-museV2-RESCUE-museV2 #PWR115
+L GND-RESCUE-museV2-RESCUE-museV2 #PWR0104
 U 1 1 57E8147A
 P 3950 3250
-F 0 "#PWR115" H 3950 3000 50  0001 C CNN
+F 0 "#PWR0104" H 3950 3000 50  0001 C CNN
 F 1 "GND" H 3950 3100 50  0000 C CNN
 F 2 "" H 3950 3250 50  0000 C CNN
@@
 $EndComp
 $Comp
-L +1.8VSB #PWR112
+L +1.8VSB #PWR0105
 U 1 1 57E81499
 P 3450 950
-F 0 "#PWR112" H 3450 1090 20  0001 C CNN
+F 0 "#PWR0105" H 3450 1090 20  0001 C CNN
 F 1 "+1.8VSB" H 3450 1060 30  0000 C CNN
 F 2 "" H 3450 950 60  0000 C CNN
@@
 F 0 "U19" H 3750 1350 60  0000 C CNN
 F 1 "GTL2010" H 4200 -400 60  0000 C CNN
-F 2 "" H 3500 1350 60  0001 C CNN
+F 2 "Housings_SSOP:SSOP-24_5.3x8.2mm_Pitch0.65mm" H 3500 1350 60  0001 C CNN
 F 3 "" H 3500 1350 60  0001 C CNN
 	1    3700 1300
@@
 $EndComp
 $Comp
-L GND-RESCUE-museV2-RESCUE-museV2 #PWR114
+L GND-RESCUE-museV2-RESCUE-museV2 #PWR0106
 U 1 1 57EB13B0
 P 4450 1850
-F 0 "#PWR114" H 4450 1850 30  0001 C CNN
+F 0 "#PWR0106" H 4450 1850 30  0001 C CNN
 F 1 "GND" H 4450 1780 30  0001 C CNN
 F 2 "" H 4450 1850 60  0000 C CNN
@@
 $EndComp
 $Comp
-L GND-RESCUE-museV2-RESCUE-museV2 #PWR119
+L GND-RESCUE-museV2-RESCUE-museV2 #PWR0107
 U 1 1 57EB2692
 P 3950 6050
-F 0 "#PWR119" H 3950 5800 50  0001 C CNN
+F 0 "#PWR0107" H 3950 5800 50  0001 C CNN
 F 1 "GND" H 3950 5900 50  0000 C CNN
 F 2 "" H 3950 6050 50  0000 C CNN
@@
 $EndComp
 $Comp
-L +1.8VSB #PWR116
+L +1.8VSB #PWR0108
 U 1 1 57EB2698
 P 3450 3750
-F 0 "#PWR116" H 3450 3890 20  0001 C CNN
+F 0 "#PWR0108" H 3450 3890 20  0001 C CNN
 F 1 "+1.8VSB" H 3450 3860 30  0000 C CNN
 F 2 "" H 3450 3750 60  0000 C CNN
@@
 $EndComp
 $Comp
-L +5VSB #PWR117
+L +5VSB #PWR0109
 U 1 1 57EB26EB
 P 4450 3750
-F 0 "#PWR117" H 4450 3840 20  0001 C CNN
+F 0 "#PWR0109" H 4450 3840 20  0001 C CNN
 F 1 "+5VSB" H 4450 3850 30  0000 C CNN
 F 2 "" H 4450 3750 60  0000 C CNN
@@
 F 0 "U20" H 3750 4150 60  0000 C CNN
 F 1 "GTL2010" H 4200 2400 60  0000 C CNN
-F 2 "" H 3500 4150 60  0001 C CNN
+F 2 "Housings_SSOP:SSOP-24_5.3x8.2mm_Pitch0.65mm" H 3500 4150 60  0001 C CNN
 F 3 "" H 3500 4150 60  0001 C CNN
 	1    3700 4100
@@
 $EndComp
 $Comp
-L GND-RESCUE-museV2-RESCUE-museV2 #PWR118
+L GND-RESCUE-museV2-RESCUE-museV2 #PWR0110
 U 1 1 57EB27CC
 P 4450 4650
-F 0 "#PWR118" H 4450 4650 30  0001 C CNN
+F 0 "#PWR0110" H 4450 4650 30  0001 C CNN
 F 1 "GND" H 4450 4580 30  0001 C CNN
 F 2 "" H 4450 4650 60  0000 C CNN
@@
 $EndComp
 $Comp
-L +3.3VSB #PWR113
+L +3.3VSB #PWR0111
 U 1 1 57EB2AFA
 P 4450 950
-F 0 "#PWR113" H 4450 910 30  0001 C CNN
+F 0 "#PWR0111" H 4450 910 30  0001 C CNN
 F 1 "+3.3VSB" H 4450 1060 30  0000 C CNN
 F 2 "" H 4450 950 60  0000 C CNN
@@
 $EndComp
 $Comp
-L GND-RESCUE-museV2-RESCUE-museV2 #PWR125
+L GND-RESCUE-museV2-RESCUE-museV2 #PWR0112
 U 1 1 57EB2FFD
 P 3950 8950
-F 0 "#PWR125" H 3950 8700 50  0001 C CNN
+F 0 "#PWR0112" H 3950 8700 50  0001 C CNN
 F 1 "GND" H 3950 8800 50  0000 C CNN
 F 2 "" H 3950 8950 50  0000 C CNN
@@
 F 0 "U21" H 3750 7050 60  0000 C CNN
 F 1 "GTL2010" H 4200 5300 60  0000 C CNN
-F 2 "" H 3500 7050 60  0001 C CNN
+F 2 "Housings_SSOP:SSOP-24_5.3x8.2mm_Pitch0.65mm" H 3500 7050 60  0001 C CNN
 F 3 "" H 3500 7050 60  0001 C CNN
 	1    3700 7000
@@
 $EndComp
 $Comp
-L +5VSB #PWR123
+L +5VSB #PWR0113
 U 1 1 5800A98D
 P 4450 6650
-F 0 "#PWR123" H 4450 6740 20  0001 C CNN
+F 0 "#PWR0113" H 4450 6740 20  0001 C CNN
 F 1 "+5VSB" H 4450 6750 30  0000 C CNN
 F 2 "" H 4450 6650 60  0000 C CNN
@@
 $EndComp
 $Comp
-L GND-RESCUE-museV2-RESCUE-museV2 #PWR124
+L GND-RESCUE-museV2-RESCUE-museV2 #PWR0114
 U 1 1 5800AA0C
 P 4450 7550
-F 0 "#PWR124" H 4450 7550 30  0001 C CNN
+F 0 "#PWR0114" H 4450 7550 30  0001 C CNN
 F 1 "GND" H 4450 7480 30  0001 C CNN
 F 2 "" H 4450 7550 60  0000 C CNN
@@
 LVL_SHIFT_4
 $Comp
-L +1.8VSB #PWR122
+L +1.8VSB #PWR0115
 U 1 1 5800ACCE
 P 3450 6650
-F 0 "#PWR122" H 3450 6790 20  0001 C CNN
+F 0 "#PWR0115" H 3450 6790 20  0001 C CNN
 F 1 "+1.8VSB" H 3450 6760 30  0000 C CNN
 F 2 "" H 3450 6650 60  0000 C CNN
@@
 Connection ~ 5600 7150
 $Comp
-L +5VSB #PWR121
+L +5VSB #PWR0116
 U 1 1 58010FD6
 P 6650 6500
-F 0 "#PWR121" H 6650 6590 20  0001 C CNN
+F 0 "#PWR0116" H 6650 6590 20  0001 C CNN
 F 1 "+5VSB" H 6650 6650 55  0000 C CNN
 F 2 "" H 6650 6500 60  0000 C CNN
@@
 $EndComp
 $Comp
-L +3.3VSB #PWR120
+L +3.3VSB #PWR0117
 U 1 1 5801107C
 P 5600 6500
-F 0 "#PWR120" H 5600 6460 30  0001 C CNN
+F 0 "#PWR0117" H 5600 6460 30  0001 C CNN
 F 1 "+3.3VSB" H 5600 6650 55  0000 C CNN
 F 2 "" H 5600 6500 60  0000 C CNN
