File: Hardware/AUDIO_ICS.sch (KiCad schematic (older format))
At the start: 44 parts, among them U10 PCM1863, U9 PCM9211, X1 24.576 MHz

Commit message: Added proper audio connectors to schematic
Parts:
- U10: footprint (none) -> muse-v2-lib:TSSOP-30_4.1x7.8mm_Pitch0.5mm
- U9: footprint (none) -> Housings_QFP:LQFP-48_7x7mm_Pitch0.5mm
Changed lines of the file:
@@
 ADC unused\nAnalog VCC\nGrounded
 $Comp
-L +3.3VSB #PWR40
+L +3.3VSB #PWR039
 U 1 1 57F2FC3A
 P 2950 1300
-F 0 "#PWR40" H 2950 1260 30  0001 C CNN
+F 0 "#PWR039" H 2950 1260 30  0001 C CNN
 F 1 "+3.3VSB" H 2950 1400 30  0000 C CNN
 F 2 "" H 2950 1300 60  0000 C CNN
@@
 Pulled LOW for\nI2C mode
 $Comp
-L GND-RESCUE-museV2-RESCUE-museV2 #PWR42
+L GND-RESCUE-museV2-RESCUE-museV2 #PWR040
 U 1 1 57F2FC41
 P 2950 2250
-F 0 "#PWR42" H 2950 2250 30  0001 C CNN
+F 0 "#PWR040" H 2950 2250 30  0001 C CNN
 F 1 "GND" H 2950 2180 30  0001 C CNN
 F 2 "" H 2950 2250 60  0000 C CNN
@@
 $EndComp
 $Comp
-L GND-RESCUE-museV2-RESCUE-museV2 #PWR49
+L GND-RESCUE-museV2-RESCUE-museV2 #PWR041
 U 1 1 57F2FC5D
 P 2100 5250
-F 0 "#PWR49" H 2100 5250 30  0001 C CNN
+F 0 "#PWR041" H 2100 5250 30  0001 C CNN
 F 1 "GND" H 2100 5180 30  0001 C CNN
 F 2 "" H 2100 5250 60  0000 C CNN
@@
 $EndComp
 $Comp
-L GND-RESCUE-museV2-RESCUE-museV2 #PWR48
+L GND-RESCUE-museV2-RESCUE-museV2 #PWR042
 U 1 1 57F2FC6A
 P 5700 5100
-F 0 "#PWR48" H 5700 5100 30  0001 C CNN
+F 0 "#PWR042" H 5700 5100 30  0001 C CNN
 F 1 "GND" H 5700 5030 30  0001 C CNN
 F 2 "" H 5700 5100 60  0000 C CNN
@@
 $EndComp
 $Comp
-L GND-RESCUE-museV2-RESCUE-museV2 #PWR47
+L GND-RESCUE-museV2-RESCUE-museV2 #PWR043
 U 1 1 57F2FC77
 P 5450 5100
-F 0 "#PWR47" H 5450 5100 30  0001 C CNN
+F 0 "#PWR043" H 5450 5100 30  0001 C CNN
 F 1 "GND" H 5450 5030 30  0001 C CNN
 F 2 "" H 5450 5100 60  0000 C CNN
@@
 $EndComp
 $Comp
-L GND-RESCUE-museV2-RESCUE-museV2 #PWR46
+L GND-RESCUE-museV2-RESCUE-museV2 #PWR044
 U 1 1 57F2FC84
 P 5300 5100
-F 0 "#PWR46" H 5300 5100 30  0001 C CNN
+F 0 "#PWR044" H 5300 5100 30  0001 C CNN
 F 1 "GND" H 5300 5030 30  0001 C CNN
 F 2 "" H 5300 5100 60  0000 C CNN
@@
 $EndComp
 $Comp
-L GND-RESCUE-museV2-RESCUE-museV2 #PWR45
+L GND-RESCUE-museV2-RESCUE-museV2 #PWR045
 U 1 1 57F2FC8A
 P 5150 5100
-F 0 "#PWR45" H 5150 5100 30  0001 C CNN
+F 0 "#PWR045" H 5150 5100 30  0001 C CNN
 F 1 "GND" H 5150 5030 30  0001 C CNN
 F 2 "" H 5150 5100 60  0000 C CNN
@@
 $EndComp
 $Comp
-L GND-RESCUE-museV2-RESCUE-museV2 #PWR44
+L GND-RESCUE-museV2-RESCUE-museV2 #PWR046
 U 1 1 57F2FC90
 P 4900 5100
-F 0 "#PWR44" H 4900 5100 30  0001 C CNN
+F 0 "#PWR046" H 4900 5100 30  0001 C CNN
 F 1 "GND" H 4900 5030 30  0001 C CNN
 F 2 "" H 4900 5100 60  0000 C CNN
@@
 F 0 "U9" H 3350 1450 60  0000 C CNN
 F 1 "PCM9211" H 4400 -1800 60  0000 C CNN
-F 2 "" H 3300 1400 60  0001 C CNN
+F 2 "Housings_QFP:LQFP-48_7x7mm_Pitch0.5mm" H 3300 1400 60  0001 C CNN
 F 3 "" H 3300 1400 60  0000 C CNN
 	1    3300 1400
@@
 $EndComp
 $Comp
-L GND-RESCUE-museV2-RESCUE-museV2 #PWR55
+L GND-RESCUE-museV2-RESCUE-museV2 #PWR047
 U 1 1 57F2FCAF
 P 2400 7600
-F 0 "#PWR55" H 2400 7600 30  0001 C CNN
+F 0 "#PWR047" H 2400 7600 30  0001 C CNN
 F 1 "GND" H 2400 7530 30  0001 C CNN
 F 2 "" H 2400 7600 60  0000 C CNN
@@
 $EndComp
 $Comp
-L GND-RESCUE-museV2-RESCUE-museV2 #PWR54
+L GND-RESCUE-museV2-RESCUE-museV2 #PWR048
 U 1 1 57F2FCB5
 P 2250 7600
-F 0 "#PWR54" H 2250 7600 30  0001 C CNN
+F 0 "#PWR048" H 2250 7600 30  0001 C CNN
 F 1 "GND" H 2250 7530 30  0001 C CNN
 F 2 "" H 2250 7600 60  0000 C CNN
@@
 $EndComp
 $Comp
-L GND-RESCUE-museV2-RESCUE-museV2 #PWR53
+L GND-RESCUE-museV2-RESCUE-museV2 #PWR049
 U 1 1 57F2FCBB
 P 2100 7600
-F 0 "#PWR53" H 2100 7600 30  0001 C CNN
+F 0 "#PWR049" H 2100 7600 30  0001 C CNN
 F 1 "GND" H 2100 7530 30  0001 C CNN
 F 2 "" H 2100 7600 60  0000 C CNN
@@
 $EndComp
 $Comp
-L GND-RESCUE-museV2-RESCUE-museV2 #PWR52
+L GND-RESCUE-museV2-RESCUE-museV2 #PWR050
 U 1 1 57F2FCC1
 P 1950 7600
-F 0 "#PWR52" H 1950 7600 30  0001 C CNN
+F 0 "#PWR050" H 1950 7600 30  0001 C CNN
 F 1 "GND" H 1950 7530 30  0001 C CNN
 F 2 "" H 1950 7600 60  0000 C CNN
@@
 $EndComp
 $Comp
-L +3.3VSB #PWR51
+L +3.3VSB #PWR051
 U 1 1 57F2FD06
 P 4150 6150
-F 0 "#PWR51" H 4150 6110 30  0001 C CNN
+F 0 "#PWR051" H 4150 6110 30  0001 C CNN
 F 1 "+3.3VSB" H 4150 6260 30  0000 C CNN
 F 2 "" H 4150 6150 60  0000 C CNN
@@
 $EndComp
 $Comp
-L +1.8VSB #PWR50
+L +1.8VSB #PWR052
 U 1 1 57F2FD0C
 P 3950 6150
-F 0 "#PWR50" H 3950 6290 20  0001 C CNN
+F 0 "#PWR052" H 3950 6290 20  0001 C CNN
 F 1 "+1.8VSB" H 3950 6260 30  0000 C CNN
 F 2 "" H 3950 6150 60  0000 C CNN
@@
 PCM1863 (ADC)
 $Comp
-L GND-RESCUE-museV2-RESCUE-museV2 #PWR62
+L GND-RESCUE-museV2-RESCUE-museV2 #PWR053
 U 1 1 57F2FD1E
 P 5950 9700
-F 0 "#PWR62" H 5950 9700 30  0001 C CNN
+F 0 "#PWR053" H 5950 9700 30  0001 C CNN
 F 1 "GND" H 5950 9630 30  0001 C CNN
 F 2 "" H 5950 9700 60  0000 C CNN
@@
 $EndComp
 $Comp
-L GND-RESCUE-museV2-RESCUE-museV2 #PWR61
+L GND-RESCUE-museV2-RESCUE-museV2 #PWR054
 U 1 1 57F2FD2B
 P 4250 9700
-F 0 "#PWR61" H 4250 9700 30  0001 C CNN
+F 0 "#PWR054" H 4250 9700 30  0001 C CNN
 F 1 "GND" H 4250 9630 30  0001 C CNN
 F 2 "" H 4250 9700 60  0000 C CNN
@@
 $EndComp
 $Comp
-L GND-RESCUE-museV2-RESCUE-museV2 #PWR59
+L GND-RESCUE-museV2-RESCUE-museV2 #PWR055
 U 1 1 57F2FD4E
 P 2400 9700
-F 0 "#PWR59" H 2400 9700 30  0001 C CNN
+F 0 "#PWR055" H 2400 9700 30  0001 C CNN
 F 1 "GND" H 2400 9630 30  0001 C CNN
 F 2 "" H 2400 9700 60  0000 C CNN
@@
 $EndComp
 $Comp
-L GND-RESCUE-museV2-RESCUE-museV2 #PWR58
+L GND-RESCUE-museV2-RESCUE-museV2 #PWR056
 U 1 1 57F2FD54
 P 2250 9700
-F 0 "#PWR58" H 2250 9700 30  0001 C CNN
+F 0 "#PWR056" H 2250 9700 30  0001 C CNN
 F 1 "GND" H 2250 9630 30  0001 C CNN
 F 2 "" H 2250 9700 60  0000 C CNN
@@
 $EndComp
 $Comp
-L GND-RESCUE-museV2-RESCUE-museV2 #PWR57
+L GND-RESCUE-museV2-RESCUE-museV2 #PWR057
 U 1 1 57F2FD5A
 P 2100 9700
-F 0 "#PWR57" H 2100 9700 30  0001 C CNN
+F 0 "#PWR057" H 2100 9700 30  0001 C CNN
 F 1 "GND" H 2100 9630 30  0001 C CNN
 F 2 "" H 2100 9700 60  0000 C CNN
@@
 $EndComp
 $Comp
-L GND-RESCUE-museV2-RESCUE-museV2 #PWR56
+L GND-RESCUE-museV2-RESCUE-museV2 #PWR058
 U 1 1 57F2FD60
 P 1950 9700
-F 0 "#PWR56" H 1950 9700 30  0001 C CNN
+F 0 "#PWR058" H 1950 9700 30  0001 C CNN
 F 1 "GND" H 1950 9630 30  0001 C CNN
 F 2 "" H 1950 9700 60  0000 C CNN
@@
 F 0 "U10" H 4500 6750 60  0000 C CNN
 F 1 "PCM1863" H 5450 4500 60  0000 C CNN
-F 2 "" H 4450 6700 60  0001 C CNN
+F 2 "muse-v2-lib:TSSOP-30_4.1x7.8mm_Pitch0.5mm" H 4450 6700 60  0001 C CNN
 F 3 "" H 4450 6700 60  0000 C CNN
 	1    4450 6700
@@
 $EndComp
 $Comp
-L GND-RESCUE-museV2-RESCUE-museV2 #PWR60
+L GND-RESCUE-museV2-RESCUE-museV2 #PWR059
 U 1 1 57F2FD94
 P 3950 9700
-F 0 "#PWR60" H 3950 9700 30  0001 C CNN
+F 0 "#PWR059" H 3950 9700 30  0001 C CNN
 F 1 "GND" H 3950 9630 30  0001 C CNN
 F 2 "" H 3950 9700 60  0000 C CNN
@@
 From Edison\n(Bluetooth/\nAnalog input)
 $Comp
-L +3.3VSB #PWR43
+L +3.3VSB #PWR060
 U 1 1 57F2FDC3
 P 2950 2500
-F 0 "#PWR43" H 2950 2460 30  0001 C CNN
+F 0 "#PWR060" H 2950 2460 30  0001 C CNN
 F 1 "+3.3VSB" H 2950 2600 30  0000 C CNN
 F 2 "" H 2950 2500 60  0000 C CNN
@@
 $EndComp
 $Comp
-L GND-RESCUE-museV2-RESCUE-museV2 #PWR63
+L GND-RESCUE-museV2-RESCUE-museV2 #PWR061
 U 1 1 57F2FDC9
 P 6100 9700
-F 0 "#PWR63" H 6100 9700 30  0001 C CNN
+F 0 "#PWR061" H 6100 9700 30  0001 C CNN
 F 1 "GND" H 6100 9630 30  0001 C CNN
 F 2 "" H 6100 9700 60  0000 C CNN
@@
 Decoupling Capacitors
 $Comp
-L +1.8VSB #PWR65
+L +1.8VSB #PWR062
 U 1 1 57FA08B9
 P 2800 10250
-F 0 "#PWR65" H 2800 10390 20  0001 C CNN
+F 0 "#PWR062" H 2800 10390 20  0001 C CNN
 F 1 "+1.8VSB" H 2800 10360 30  0000 C CNN
 F 2 "" H 2800 10250 60  0000 C CNN
@@
 $EndComp
 $Comp
-L GND-RESCUE-museV2-RESCUE-museV2 #PWR67
+L GND-RESCUE-museV2-RESCUE-museV2 #PWR063
 U 1 1 57FA08BF
 P 2800 11000
-F 0 "#PWR67" H 2800 11000 30  0001 C CNN
+F 0 "#PWR063" H 2800 11000 30  0001 C CNN
 F 1 "GND" H 2800 10930 30  0001 C CNN
 F 2 "" H 2800 11000 60  0000 C CNN
@@
 $EndComp
 $Comp
-L GND-RESCUE-museV2-RESCUE-museV2 #PWR66
+L GND-RESCUE-museV2-RESCUE-museV2 #PWR064
 U 1 1 57FA08D3
 P 1900 11000
-F 0 "#PWR66" H 1900 11000 30  0001 C CNN
+F 0 "#PWR064" H 1900 11000 30  0001 C CNN
 F 1 "GND" H 1900 10930 30  0001 C CNN
 F 2 "" H 1900 11000 60  0000 C CNN
@@
 $EndComp
 $Comp
-L +3.3VSB #PWR64
+L +3.3VSB #PWR065
 U 1 1 57FA08F5
 P 1900 10250
-F 0 "#PWR64" H 1900 10210 30  0001 C CNN
+F 0 "#PWR065" H 1900 10210 30  0001 C CNN
 F 1 "+3.3VSB" H 1900 10360 30  0000 C CNN
 F 2 "" H 1900 10250 60  0000 C CNN
@@
 	2950 10300 2950 10450
 $Comp
-L GND-RESCUE-museV2-RESCUE-museV2 #PWR41
+L GND-RESCUE-museV2-RESCUE-museV2 #PWR066
 U 1 1 57FA1F81
 P 5700 1600
-F 0 "#PWR41" H 5700 1600 30  0001 C CNN
+F 0 "#PWR066" H 5700 1600 30  0001 C CNN
 F 1 "GND" H 5700 1530 30  0001 C CNN
 F 2 "" H 5700 1600 60  0000 C CNN
@@
 $EndComp
 $Comp
-L +3.3VSB #PWR39
+L +3.3VSB #PWR067
 U 1 1 57FA1FAB
 P 5700 850
-F 0 "#PWR39" H 5700 810 30  0001 C CNN
+F 0 "#PWR067" H 5700 810 30  0001 C CNN
 F 1 "+3.3VSB" H 5700 960 30  0000 C CNN
 F 2 "" H 5700 850 60  0000 C CNN
@@
 F 0 "X1" H 2580 4590 30  0000 C CNN
 F 1 "24.576 MHz" H 2730 4390 30  0000 L CNN
-F 2 "" H 2700 4500 60  0000 C CNN
+F 2 "" H 2700 4500 60  0001 C CNN
 F 3 "" H 2700 4500 60  0000 C CNN
 	1    2700 4500

Commit message: Updated libraries and place components into board layout
Parts:
- X1: footprint (none) -> muse-v2-lib:3.2x2.5mm_smd_crystal
Changed lines of the file:
@@
 F 0 "X1" H 2580 4590 30  0000 C CNN
 F 1 "24.576 MHz" H 2730 4390 30  0000 L CNN
-F 2 "" H 2700 4500 60  0001 C CNN
+F 2 "muse-v2-lib:3.2x2.5mm_smd_crystal" H 2700 4500 60  0001 C CNN
 F 3 "" H 2700 4500 60  0000 C CNN
 	1    2700 4500

Commit message: PCB Layout progress - placing PCM9211 components
Parts:
- removed C19: 0.1uF, Capacitors_SMD:C_0402, symbol C-RESCUE-museV2
- removed C81: .01uF, Capacitors_SMD:C_0402, symbol C-RESCUE-museV2
- added R6: 50, Resistors_SMD:R_0402, symbol R-RESCUE-museV2
- C15, C17, C22: footprint Capacitors_SMD:c_elec_4x4.5 -> Capacitors_SMD:C_1206
- C20, C25: value 27pF -> 15pF
- X1: footprint muse-v2-lib:3.2x2.5mm_smd_crystal -> muse-v2-lib:5x3.2mm_crystal
Connections:
- net +3.3VSB: now also C23.2, C24.2
- net GND: now also X1.4 (VDD); no longer C23.2, C24.2
- net at C25.1, X1.1 (ctl): now also R6.2; no longer U9.40 (XT0)
- new net: R6.1, U9.40 (XT0)
Other:
- note added: "Minimize oscilator traces as \nmuch as possible"
- note added: "Placement distance of\nC21, C22 not critical"
- moved on the sheet: C25
