File: Hardware/museV2.kicad_pcb (KiCad board)
At the start: 2 copper layers, 288 parts, among them P1 RCA_conn_x2, P10 -15V, P11 ~3, P13 ~4, P14 +5V, P18 RX1, P19 3.3V, P2 +12V, P20 TX2, P21 1.8V, P22 PSU_CTL, P23 GND, P27 D1, P29 D2, P3 3.5mm_conn_tip_switch, P30 D3, P31 P1, P32 L1.8_1, P33 L3.3_1, P34 P2, P35 L1.8_2, P36 L3.3_2, P37 P3, P38 L1.8_3, P39 L3.3_3, P4 3.5mm_conn_tip_switch, P40 P4, P41 L1.8_4, P42 L3.3_4, P43 +5V, P44 +12V_AUX, P45 +5V_AUX, P5 CONN_01X06, P6 CONN_02X14, P7 ~5, P8 +15V, P9 ~6, Q1 PMOS, Q2 BSS138, SW1 PWR_BTN, SW2 PWR_BTN, U1 TPS65130, U10 PCM1863, U11 PCM1796, U12 NE5534, U13 NE5534, U14 NE5534, U15 NE5534, U16 NE5534, U17 NE5534, U18 EdisonConnector, U19 GTL2010, U2 LP38692, U20 GTL2010, U21 GTL2010, U22 PCA9685BS, U3 PLR135/T10, U4 POM-3535L-3-R, U5 POM-3535L-3-R, U6 PLT133/T10W, U7 POM-3535L-3-R, U8 POM-3535L-3-R, U9 PCM9211, X1 24.576 MHz

Commit message: Placing ADC connections
Parts:
- added REF**: VIA-0.3mm, muse-v2-lib:VIA-0.3mm, F.Cu at (170.6, 137.6)
- added REF**: VIA-0.3mm, muse-v2-lib:VIA-0.3mm, F.Cu at (169.3, 138.8)
- added REF**: VIA-0.3mm, muse-v2-lib:VIA-0.3mm, F.Cu at (169.9, 137.6)
- added REF**: VIA-0.3mm, muse-v2-lib:VIA-0.3mm, F.Cu at (169.3, 138.1)
- moved C18 162.2 mm to (182.3, 166.3), turned to 0 degrees
- moved C17 132.8 mm to (183.4, 168.1), turned to 0 degrees
- moved U11 13.4 mm to (166.2, 166.7)
- moved C15 4.16 mm to (187.0, 155.8)
- moved R12 4.16 mm to (178.2, 154.1)
- moved R6 4.16 mm to (180.1, 154.1)
- moved REF** 4.16 mm to (181.4, 149.3)
- moved REF** 4.16 mm to (182.2, 151.9)
- moved REF** 4.16 mm to (181.2, 147.4)
- moved C22 4.16 mm to (171.8, 154.9)
- moved C16 4.16 mm to (185.2, 157.0)
- moved C20 4.16 mm to (183.9, 149.4)
- moved C21 4.16 mm to (175.9, 154.6)
- moved C24 4.16 mm to (172.9, 151.1)
- moved C25 4.16 mm to (177.4, 148.2)
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Routing:
- net UART_RX(1.8): track 0.00 -> 16.9 mm, vias 0 -> 2
- net UART_TX(1.8): track 0.00 -> 14.6 mm
- net I2S_MCU_DOUT(1.8): track 0.00 -> 8.21 mm, vias 0 -> 2
- net I2S_MCU_LRCK(1.8): track 0.00 -> 8.02 mm, vias 0 -> 2
- net I2S_MCU_BCK(1.8): track 0.00 -> 7.91 mm, vias 0 -> 2
- net I2S_MCU_DIN(1.8): track 0.00 -> 7.90 mm, vias 0 -> 2

Commit message: routing digital signal wires
Parts:
- removed C38: 10uF, Capacitors_SMD:c_elec_4x4.5
- removed C39: 0.1uF, Capacitors_SMD:C_0402
- removed C81: 10uF, Capacitors_SMD:C_0402
- removed the REF** at (181.4, 149.3)
- removed the REF** at (182.7, 148.4)
- removed the REF** at (182.2, 151.9)
- removed the REF** at (180.3, 151.8)
- removed the REF** at (182.6, 149.4)
- removed the REF** at (179.4, 149.2)
- removed the REF** at (178.5, 147.1)
- removed the REF** at (177.2, 147.1)
- removed the REF** at (181.2, 147.4)
- added REF**: VIA-0.3mm, muse-v2-lib:VIA-0.3mm, F.Cu at (180.1, 131.2)
- added REF**: VIA-0.3mm, muse-v2-lib:VIA-0.3mm, F.Cu at (183.2, 145.4)
- added REF**: VIA-0.3mm, muse-v2-lib:VIA-0.3mm, F.Cu at (176.8, 125.0)
- added REF**: VIA-0.3mm, muse-v2-lib:VIA-0.3mm, F.Cu at (177.8, 125.5)
- added REF**: VIA-0.3mm, muse-v2-lib:VIA-0.3mm, F.Cu at (178.6, 125.8)
- added REF**: VIA-0.3mm, muse-v2-lib:VIA-0.3mm, F.Cu at (180.2, 125.8)
- added REF**: VIA-0.3mm, muse-v2-lib:VIA-0.3mm, F.Cu at (181.6, 126.5)
- added REF**: VIA-0.3mm, muse-v2-lib:VIA-0.3mm, F.Cu at (180.2, 125.0)
- added REF**: VIA-0.3mm, muse-v2-lib:VIA-0.3mm, F.Cu at (179.4, 125.5)
- added REF**: VIA-0.3mm, muse-v2-lib:VIA-0.3mm, F.Cu at (179.6, 135.0)
- added REF**: VIA-0.3mm, muse-v2-lib:VIA-0.3mm, F.Cu at (178.6, 125.0)
- added REF**: VIA-0.3mm, muse-v2-lib:VIA-0.3mm, F.Cu at (183.9, 145.4)
- added REF**: VIA-0.3mm, muse-v2-lib:VIA-0.3mm, F.Cu at (186.6, 132.7)
- added REF**: VIA-0.3mm, muse-v2-lib:VIA-0.3mm, F.Cu at (180.4, 135.0)
- added REF**: VIA-0.3mm, muse-v2-lib:VIA-0.3mm, F.Cu at (188.2, 129.6)
- added REF**: VIA-0.3mm, muse-v2-lib:VIA-0.3mm, F.Cu at (187.3, 129.6)
- added REF**: VIA-0.3mm, muse-v2-lib:VIA-0.3mm, F.Cu at (186.6, 130.2)
- added REF**: VIA-0.3mm, muse-v2-lib:VIA-0.3mm, F.Cu at (186.6, 131.1)
- added REF**: VIA-0.3mm, muse-v2-lib:VIA-0.3mm, F.Cu at (186.6, 131.8)
- added REF**: VIA-0.3mm, muse-v2-lib:VIA-0.3mm, F.Cu at (181.8, 144.7)
- added REF**: VIA-0.3mm, muse-v2-lib:VIA-0.3mm, F.Cu at (182.4, 145.4)
- C15, C17, C40: moved to B.Cu
- C36, C47: footprint Capacitors_SMD:c_elec_4x4.5 -> Capacitors_SMD:C_1206; moved to B.Cu
- moved C48 187.4 mm to (170.4, 128.3), turned to 270 degrees
- moved C47 179.5 mm to (168.9, 128.3)
- moved C37 159.2 mm to (168.3, 144.5), turned to 0 degrees
- moved C41 152.0 mm to (166.6, 145.1), turned to 90 degrees
- moved C36 130.8 mm to (167.8, 144.6), turned to 270 degrees
- moved C40 128.3 mm to (165.9, 143.8), turned to 270 degrees
- moved U11 37.3 mm to (165.1, 129.3)
- moved C17 35.8 mm to (181.5, 132.3), turned to 90 degrees
- moved C18 32.3 mm to (180.8, 134.1), turned to 180 degrees
- moved R12 32.3 mm to (176.9, 121.8), turned to 90 degrees
- moved C21 32.3 mm to (174.7, 122.2)
- moved C20 32.3 mm to (183.2, 117.1)
- moved C24 32.3 mm to (172.2, 118.8)
- moved C25 32.3 mm to (176.8, 115.8)
- moved U9 32.3 mm to (178.7, 128.2)
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Connections:
- C42 pad 1: +5VSB -> +5V
- C43 pad 1: +5VSB -> +5V
- C44 pad 1: +5VSB -> +5V
- C45 pad 1: +5VSB -> +5V
- C46 pad 1: +5VSB -> +5V
- C49 pad 1: +5VSB -> +5V
- P11 pad 1: (no net) -> MCU_GPIO_X_3/PWM_X_3
- P13 pad 1: (no net) -> MCU_GPIO_X_4/PWM_X_4
- P45 pad 1: (no net) -> +5V
- P5 pad 3: (no net) -> Net-(P5-Pad3)
- P5 pad 6: (no net) -> Net-(P5-Pad6)
- P6 pad 5: (no net) -> /LIGHT_CONN/LED_B_1
- P7 pad 1: (no net) -> MCU_GPIO_X_5/PWM_X_1
- P9 pad 1: (no net) -> MCU_GPIO_X_6/PWM_X_2
- U1 pad 12: (no net) -> Net-(U1-Pad12)
- U1 pad 20: (no net) -> Net-(U1-Pad20)
- U1 pad 25: GND -> (no net)
- U10 pad 10: (no net) -> Net-(U10-Pad10)
- U10 pad 19: (no net) -> Net-(U10-Pad19)
- U10 pad 22: (no net) -> Net-(U10-Pad22)
- U10 pad 9: (no net) -> Net-(U10-Pad9)
- U11 pad 1: (no net) -> Net-(U11-Pad1)
- U11 pad 15: +5VSB -> +5V
- U11 pad 2: (no net) -> Net-(U11-Pad2)
- U11 pad 23: +5VSB -> +5V
- U11 pad 28: +5VSB -> +5V
- U18 pad 10: (no net) -> Net-(U18-Pad10)
- U18 pad 16: (no net) -> Net-(U18-Pad16)
- U18 pad 18: (no net) -> Net-(U18-Pad18)
- U18 pad 19: (no net) -> Net-(U18-Pad19)
- U18 pad 20: (no net) -> Net-(U18-Pad20)
- U18 pad 21: (no net) -> Net-(U18-Pad21)
- U18 pad 23: (no net) -> Net-(U18-Pad23)
- U18 pad 24: (no net) -> Net-(U18-Pad24)
- U18 pad 3: (no net) -> Net-(U18-Pad3)
- U18 pad 31: (no net) -> Net-(U18-Pad31)
- U18 pad 33: (no net) -> MCU_GPIO_X_4/PWM_X_2
- U18 pad 35: (no net) -> MCU_GPIO_X_3/PWM_X_1
- U18 pad 37: (no net) -> MCU_GPIO_X_5/PWM_X_3
- U18 pad 39: (no net) -> MCU_GPIO_X_6/PWM_X_4
- U18 pad 67: (no net) -> Net-(U18-Pad67)
- U18 pad 69: (no net) -> Net-(U18-Pad69)
- U18 pad 7: (no net) -> Net-(U18-Pad7)
- U18 pad 8: (no net) -> Net-(U18-Pad8)
- U9 pad 1: (no net) -> Net-(U9-Pad1)
- U9 pad 16: (no net) -> Net-(U9-Pad16)
- U9 pad 2: (no net) -> Net-(U9-Pad2)
- U9 pad 32: (no net) -> Net-(U9-Pad32)
- U9 pad 35: (no net) -> Net-(U9-Pad35)
- U9 pad 37: (no net) -> Net-(U9-Pad37)
- U9 pad 47: (no net) -> Net-(U9-Pad47)
- U9 pad 48: (no net) -> Net-(U9-Pad48)
Routing:
- net ADC_CLKE_INT: track 0.00 -> 36.5 mm, vias 0 -> 4
- net I2C_SCL(3.3): track 1.88 -> 35.4 mm, vias 0 -> 6
- net I2C_SDA(3.3): track 0.00 -> 32.0 mm, vias 0 -> 4
- net I2S_SCK(3.3): track 0.00 -> 20.8 mm
- net I2S_MCU_BCK(3.3): track 3.68 -> 23.2 mm, vias 0 -> 4
- net I2S_MCU_LRCK(3.3): track 3.68 -> 22.2 mm, vias 0 -> 2
- net I2S_SCK: track 0.00 -> 15.7 mm, vias 0 -> 2
- net I2S_ADC_DOUT: track 0.00 -> 12.3 mm
- net I2S_ADC_BCK: track 0.00 -> 9.93 mm, vias 0 -> 2
- net I2S_MCU_DIN(3.3): track 3.95 -> 13.3 mm
- net I2S_ADC_LRCK: track 0.00 -> 9.05 mm
- net Net-(C24-Pad1): track 10.8 -> 3.09 mm
- net BT_PAIR_BTN: track 0.00 -> 7.35 mm, vias 0 -> 2
- net I2S_DAC_LRCK(3.3): track 0.00 -> 6.50 mm
- net I2S_DAC_BCK(3.3): track 0.00 -> 6.17 mm
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- added copper zone on F.Cu, net I2C_SCL(3.3)
