File: Hardware/_autosave-museV2.kicad_pcb (KiCad board)
At the start: 2 copper layers, 352 parts, among them P1 RCA_conn_x2, P10 -15V, P11 ~4, P12 1, P13 ~5, P14 +5V, P18 RX7, P19 3.3V, P2 +12V, P20 TX6, P21 1.8V, P22 PSU_CTL, P23 GND, P27 D1, P29 D2, P3 3.5mm_conn_tip_switch, P30 D3, P31 P1, P32 L1.8_1, P33 L3.3_1, P34 P2, P35 L1.8_2, P36 L3.3_2, P37 P3, P38 L1.8_3, P39 L3.3_3, P4 3.5mm_conn_tip_switch, P40 P4, P41 L1.8_4, P42 L3.3_4, P43 +5V, P44 +12V_AUX, P45 +5V_AUX, P5 CONN_01X06, P6 CONN_02X14, P7 ~2, P8 +15V, P9 ~3, Q1 PMOS, Q2 BSS138, SW1 PWR_BTN, SW2 PWR_BTN, U1 TPS65130, U10 PCM1863, U11 PCM1796, U12 NE5534, U13 NE5534, U14 NE5534, U15 NE5534, U16 NE5534, U17 NE5534, U18 EdisonConnector, U19 GTL2010, U2 LP38692, U20 GTL2010, U21 GTL2010, U22 PCA9685BS, U3 PLR135/T10, U4 POM-3535L-3-R, U5 POM-3535L-3-R, U6 PLT133/T10W, U7 POM-3535L-3-R, U8 POM-3535L-3-R, U9 PCM9211, X1 24.576 MHz

Commit message: Completed placement of level shifters
Parts:
- moved R65 6.46 mm to (226.2, 129.7), turned to 180 degrees
- moved R111 5.87 mm to (233.2, 132.4)
- moved R86 5.76 mm to (226.2, 139.8), turned to 180 degrees
- moved C80 3.95 mm to (226.3, 141.9)
- moved R108 3.95 mm to (224.2, 140.7)
- moved REF** 3.95 mm to (227.4, 140.8)
- moved REF** 3.95 mm to (227.9, 142.1)
- moved REF** 3.95 mm to (226.8, 140.8)
- moved U21 3.95 mm to (216.6, 141.4)
- moved R105 3.95 mm to (222.1, 137.8)
- moved R106 3.95 mm to (223.4, 137.8)
- moved R107 3.95 mm to (224.2, 139.4)
- moved R109 3.95 mm to (224.2, 142.0)
- moved R110 3.95 mm to (224.2, 143.3)
- moved R87 3.95 mm to (213.7, 148.1)
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Routing:
- net I2C_PWM_SDA(3.3): track 61.5 -> 60.5 mm
- net LED_IA_11(1.8): track 22.6 -> 23.2 mm
Other:
- net class Default: trace_width 0.45 -> 0.25

Commit message: Digital Half completed placement
Parts:
- removed P12: 1, Pin_Headers:Pin_Header_Straight_1x01
- removed P14: +5V, Pin_Headers:Pin_Header_Straight_1x01
- removed P2: +12V, Pin_Headers:Pin_Header_Straight_1x01
- removed P27: D1, Pin_Headers:Pin_Header_Straight_1x01
- removed P29: D2, Pin_Headers:Pin_Header_Straight_1x01
- removed P30: D3, Pin_Headers:Pin_Header_Straight_1x01
- removed P44: +12V_AUX, Pin_Headers:Pin_Header_Straight_1x01
- removed P45: +5V_AUX, Pin_Headers:Pin_Header_Straight_1x01
- removed the REF** at (227.9, 141.4)
- removed the REF** at (227.9, 142.1)
- added C39: 2.2uF, Capacitors_SMD:C_0402, F.Cu at (104.6, 144.1)
- added C81: 2.2uF, Capacitors_SMD:C_0402, F.Cu at (104.8, 137.4)
- added C82: 2.2uF, Capacitors_SMD:C_0402, F.Cu at (104.9, 140.7)
- added C83: 2.2uF, Capacitors_SMD:C_0402, F.Cu at (104.8, 134.2)
- added C84: 2.2uF, Capacitors_SMD:C_0402, F.Cu at (107.7, 134.2)
- added C85: 2.2uF, Capacitors_SMD:C_0402, F.Cu at (107.5, 137.7)
- added C86: 2.2uF, Capacitors_SMD:C_0402, F.Cu at (107.7, 141.0)
- added C87: 2.2uF, Capacitors_SMD:C_0402, F.Cu at (107.6, 144.2)
- added C88: 2.2uF, Capacitors_SMD:C_0402, F.Cu at (107.5, 147.7)
- added C89: 2.2uF, Capacitors_SMD:C_0402, F.Cu at (104.7, 147.5)
- added C90: 2.2uF, Capacitors_SMD:C_0402, F.Cu at (107.5, 151.1)
- added C91: 2.2uF, Capacitors_SMD:C_0402, F.Cu at (104.7, 151.3)
- added REF**: VIA-0.3mm, muse-v2-lib:VIA-0.3mm, F.Cu at (211.5, 137.7)
- added REF**: VIA-0.3mm, muse-v2-lib:VIA-0.3mm, F.Cu at (213.4, 125.5)
- added REF**: VIA-0.3mm, muse-v2-lib:VIA-0.3mm, F.Cu at (212.5, 125.5)
- added REF**: VIA-0.3mm, muse-v2-lib:VIA-0.3mm, F.Cu at (213.4, 137.1)
- added REF**: VIA-0.3mm, muse-v2-lib:VIA-0.3mm, F.Cu at (212.4, 137.1)
- added REF**: VIA-0.3mm, muse-v2-lib:VIA-0.3mm, F.Cu at (160.6, 100.2)
- added REF**: VIA-0.3mm, muse-v2-lib:VIA-0.3mm, F.Cu at (161.5, 100.1)
- added REF**: VIA-0.3mm, muse-v2-lib:VIA-0.3mm, F.Cu at (160.6, 101.0)
- added REF**: VIA-0.3mm, muse-v2-lib:VIA-0.3mm, F.Cu at (166.9, 98.3)
- added REF**: VIA-0.3mm, muse-v2-lib:VIA-0.3mm, F.Cu at (165.8, 98.3)
- added REF**: VIA-0.3mm, muse-v2-lib:VIA-0.3mm, F.Cu at (211.6, 126.0)
- added REF**: VIA-0.3mm, muse-v2-lib:VIA-0.3mm, F.Cu at (165.1, 99.0)
- C13, C14, R100, R101, R102, R103, R104, R113, R114, R115, R116, R117, R118, R45, R46, R47, R48, R49, R50, R51, R52, R53, R54, R66, R67, R68, R69, R70, R71, R72, R73, R74, R75, R95, R96, R97, R98, R99: moved to B.Cu
- SW2: value PWR_BTN -> PAIR_BTN
- moved P43 130.3 mm to (156.6, 97.5), turned to 90 degrees
- moved P22 120.3 mm to (160.1, 97.5)
- moved P23 117.5 mm to (156.6, 101.1), turned to 90 degrees
- moved R68 115.1 mm to (213.1, 129.7), turned to 0 degrees
- moved R73 110.8 mm to (213.1, 134.8), turned to 0 degrees
- moved P8 109.0 mm to (155.8, 110.3)
- moved R67 108.8 mm to (213.1, 128.3), turned to 0 degrees
- moved R69 107.3 mm to (213.1, 130.9), turned to 0 degrees
- moved R96 106.8 mm to (201.2, 141.8), turned to 270 degrees
- moved R74 106.4 mm to (197.6, 138.9), turned to 270 degrees
- moved R72 105.9 mm to (213.1, 133.6), turned to 0 degrees
- moved R75 104.8 mm to (197.2, 140.9), turned to 270 degrees
- moved R101 103.0 mm to (207.1, 146.2), turned to 90 degrees
- moved R53 102.2 mm to (183.3, 137.4)
- moved P10 99.8 mm to (169.3, 97.6)
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Connections:
- C42 pad 1: +5V -> +5VSB
- C43 pad 1: +5V -> +5VSB
- C44 pad 1: +5V -> +5VSB
- C45 pad 1: +5V -> +5VSB
- C46 pad 1: +5V -> +5VSB
- C49 pad 1: +5V -> +5VSB
- R113 pad 2: LED_IA_3 -> LED_IA_11
- R114 pad 2: LED_IA_4 -> LED_IA_12
- R115 pad 2: LED_IA_5 -> LED_IA_13
- R116 pad 2: LED_IA_6 -> LED_IA_14
- R117 pad 2: LED_IA_7 -> LED_IA_15
- R118 pad 2: LED_IA_8 -> LED_IA_16
- R119 pad 2: LED_IA_9 -> LED_IA_3
- R120 pad 2: LED_IA_10 -> LED_IA_4
- R121 pad 2: LED_IA_11 -> LED_IA_5
- R122 pad 2: LED_IA_12 -> LED_IA_6
- R123 pad 2: LED_IA_13 -> LED_IA_7
- R124 pad 2: LED_IA_14 -> LED_IA_8
- R125 pad 2: LED_IA_15 -> LED_IA_9
- R126 pad 2: LED_IA_16 -> LED_IA_10
- U11 pad 15: +5V -> +5VSB
- U11 pad 23: +5V -> +5VSB
- U11 pad 28: +5V -> +5VSB
- U18 pad 25: MCU_GPIO_X_1 -> Net-(U18-Pad25)
- U9 pad 4: DFE_GPIO_X_1 -> Net-(U9-Pad4)
- U9 pad 5: DFE_GPIO_X_2 -> Net-(U9-Pad5)
- U9 pad 6: DFE_GPIO_X_3 -> Net-(U9-Pad6)
Routing:
- net PSU_CTL: track 0.00 -> 100.0 mm, vias 0 -> 6
- net MCU_GPIO_X_4/PWM_X_3: track 0.00 -> 75.9 mm, vias 0 -> 6
- net MCU_GPIO_X_3/PWM_X_2: track 0.00 -> 70.7 mm, vias 0 -> 6
- net MCU_GPIO_X_2/PWM_X_1: track 0.00 -> 66.6 mm, vias 0 -> 6
- net LED_IA_9: track 3.61 -> 67.8 mm, vias 0 -> 2
- net LED_IA_10: track 1.70 -> 65.6 mm, vias 0 -> 2
- net LED_IA_8: track 4.62 -> 67.7 mm, vias 0 -> 2
- net LED_IA_7: track 4.29 -> 65.6 mm, vias 0 -> 2
- net LED_IA_11: track 2.26 -> 60.4 mm, vias 0 -> 1
- net MCU_GPIO_X_6/UART_TX: track 0.00 -> 57.1 mm, vias 0 -> 2
- net LED_IA_6: track 4.02 -> 58.9 mm, vias 0 -> 2
- net LED_IA_5: track 3.75 -> 56.9 mm, vias 0 -> 2
- net LED_IA_12: track 3.83 -> 55.2 mm, vias 0 -> 1
- net LED_IA_4: track 3.71 -> 52.6 mm, vias 0 -> 2
- net LED_IA_13: track 3.97 -> 51.8 mm, vias 0 -> 1
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Other:
- board outline added: 142.3 x 55.5 mm
