File: Hardware/_autosave-museV2.kicad_pcb (KiCad board)
At the start: 2 copper layers, 142.3 x 55.5 mm, 391 parts, among them P1 RCA_conn_x2, P10 -15V, P11 ~4, P13 ~5, P18 RX7, P19 3.3V, P20 TX6, P21 1.8V, P22 PSU_CTL, P23 GND, P3 3.5mm_conn_tip_switch, P31 P1, P32 L1.8_1, P33 L3.3_1, P34 P2, P35 L1.8_2, P36 L3.3_2, P37 P3, P38 L1.8_3, P39 L3.3_3, P4 3.5mm_conn_tip_switch, P40 P4, P41 L1.8_4, P42 L3.3_4, P43 +5V, P5 CONN_01X06, P6 CONN_02X14, P7 ~2, P8 +15V, P9 ~3, Q1 PMOS, Q2 BSS138, SW1 PWR_BTN, SW2 PAIR_BTN, U1 TPS65130, U10 PCM1863, U11 PCM1796, U12 NE5534, U13 NE5534, U14 NE5534, U15 NE5534, U16 NE5534, U17 NE5534, U18 EdisonConnector, U19 GTL2010, U2 LP38692, U20 GTL2010, U21 GTL2010, U22 PCA9685BS, U3 PLR135/T10, U4 POM-3535L-3-R, U5 POM-3535L-3-R, U6 PLT133/T10W, U7 POM-3535L-3-R, U8 POM-3535L-3-R, U9 PCM9211, X1 24.576 MHz

Commit message: Op-Amp placement and wiring
Parts:
- removed C39, C89, C90, C91: 2.2uF, Capacitors_SMD:c_elec_4x5.3
- added R129: 22K, Resistors_SMD:R_0402, F.Cu at (168.7, 165.2)
- added R130: 22K, Resistors_SMD:R_0402, F.Cu at (146.2, 134.1)
- added R131: 22K, Resistors_SMD:R_0402, F.Cu at (146.7, 122.5)
- added R132: 22K, Resistors_SMD:R_0402, F.Cu at (168.4, 161.2)
- added R133: 22K, Resistors_SMD:R_0402, F.Cu at (146.7, 111.0)
- added R134: 0, Resistors_SMD:R_0402, F.Cu at (154.5, 142.6)
- added R135: 0, Resistors_SMD:R_0402, F.Cu at (152.0, 141.4)
- added R136: 0, Resistors_SMD:R_0402, F.Cu at (164.3, 153.7)
- added R137: 0, Resistors_SMD:R_0402, F.Cu at (168.3, 153.6)
- added R138: 0, Resistors_SMD:R_0402, F.Cu at (172.4, 153.7)
- added R139: 0, Resistors_SMD:R_0402, F.Cu at (176.3, 153.7)
- added R140: 0, Resistors_SMD:R_0402, F.Cu at (164.3, 172.2)
- added R141: 0, Resistors_SMD:R_0402, F.Cu at (164.3, 161.1)
- added R7: 22K, Resistors_SMD:R_0402, F.Cu at (146.7, 145.4)
- added RV1: 100K, muse-v2-lib:TC33X-1, F.Cu at (146.6, 148.4)
- added RV2: 100K, muse-v2-lib:TC33X-1, F.Cu at (177.8, 160.8)
- added RV3: 100K, muse-v2-lib:TC33X-1, F.Cu at (146.6, 136.9)
- added RV4: 100K, muse-v2-lib:TC33X-1, F.Cu at (146.6, 125.5)
- added RV5: 100K, muse-v2-lib:TC33X-1, F.Cu at (177.8, 169.0)
- added RV6: 100K, muse-v2-lib:TC33X-1, F.Cu at (146.6, 114.0)
- C81, C84, C85, C88: value 2.2uF -> 4.7uF; moved to B.Cu
- moved C52 85.5 mm to (150.1, 103.8), turned to 90 degrees
- moved C54 80.4 mm to (142.4, 108.3)
- moved C83 74.0 mm to (180.8, 175.8)
- moved C88 72.9 mm to (143.9, 121.0), turned to 180 degrees
- moved C85 72.2 mm to (154.3, 118.5), turned to 180 degrees
- moved C51 71.9 mm to (152.2, 117.2), turned to 0 degrees
- moved C82 65.8 mm to (172.8, 175.8)
- moved U17 64.9 mm to (147.3, 107.7)
- moved U14 63.6 mm to (147.3, 130.6)
- moved C55 61.4 mm to (142.4, 119.8)
- moved C81 60.8 mm to (154.3, 137.1), turned to 180 degrees
- moved C50 56.1 mm to (152.9, 143.3), turned to 90 degrees
- moved U12 52.6 mm to (147.3, 142.0)
- moved C84 48.7 mm to (143.9, 137.1), turned to 180 degrees
- moved C87 48.6 mm to (156.5, 168.7)
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Connections:
- C50 pad 2: /DAC/sheet57F8A4E6/ANALOG_OUT- -> Net-(C50-Pad2)
- C60 pad 2: /DAC/sheet57F8A4E6/ANALOG_OUT+ -> Net-(C60-Pad2)
- C64 pad 2: /DAC/sheet57F8A4E7/ANALOG_OUT- -> Net-(C64-Pad2)
- C74 pad 2: /DAC/sheet57F8A4E7/ANALOG_OUT+ -> Net-(C74-Pad2)
- C81 pad 1: -15V -> GND
- C81 pad 2: GND -> -15V
- C82 pad 1: -15V -> GND
- C82 pad 2: GND -> -15V
- C85 pad 1: +15V -> GND
- C85 pad 2: GND -> -15V
- C86 pad 1: -15V -> GND
- C86 pad 2: GND -> -15V
- C87 pad 1: -15V -> +15V
- C88 pad 1: -15V -> +15V
- R26 pad 2: /DAC/sheet57F8A4E6/ANALOG_OUT- -> Net-(C50-Pad2)
- R33 pad 2: /DAC/sheet57F8A4E6/ANALOG_OUT+ -> Net-(C60-Pad2)
- R35 pad 2: /DAC/sheet57F8A4E7/ANALOG_OUT- -> Net-(C64-Pad2)
- R42 pad 2: /DAC/sheet57F8A4E7/ANALOG_OUT+ -> Net-(C74-Pad2)
- U12 pad 1: (no net) -> Net-(RV1-Pad3)
- U12 pad 2: /DAC/sheet57F8A4E6/ANALOG_OUT- -> Net-(C50-Pad2)
- U12 pad 3: GND -> Net-(R135-Pad1)
- U12 pad 5: Net-(C57-Pad1) -> Net-(C57-Pad2)
- U12 pad 8: Net-(C57-Pad2) -> Net-(C57-Pad1)
- U13 pad 1: (no net) -> Net-(RV2-Pad3)
- U13 pad 5: Net-(C58-Pad1) -> Net-(C58-Pad2)
- U13 pad 8: Net-(C58-Pad2) -> Net-(C58-Pad1)
- U14 pad 1: (no net) -> Net-(RV3-Pad3)
- U14 pad 2: /DAC/sheet57F8A4E6/ANALOG_OUT+ -> Net-(C60-Pad2)
- U14 pad 3: GND -> Net-(R137-Pad1)
- U14 pad 5: Net-(C62-Pad1) -> Net-(C62-Pad2)
- U14 pad 8: Net-(C62-Pad2) -> Net-(C62-Pad1)
- U15 pad 1: (no net) -> Net-(RV4-Pad3)
- U15 pad 2: /DAC/sheet57F8A4E7/ANALOG_OUT- -> Net-(C64-Pad2)
- U15 pad 3: GND -> Net-(R139-Pad1)
- U15 pad 5: Net-(C71-Pad1) -> Net-(C71-Pad2)
- U15 pad 8: Net-(C71-Pad2) -> Net-(C71-Pad1)
- U16 pad 1: (no net) -> Net-(RV5-Pad3)
- U16 pad 5: Net-(C72-Pad1) -> Net-(C72-Pad2)
- U16 pad 8: Net-(C72-Pad2) -> Net-(C72-Pad1)
- U17 pad 1: (no net) -> Net-(RV6-Pad3)
- U17 pad 2: /DAC/sheet57F8A4E7/ANALOG_OUT+ -> Net-(C74-Pad2)
- U17 pad 3: GND -> Net-(R141-Pad1)
- U17 pad 5: Net-(C76-Pad1) -> Net-(C76-Pad2)
- U17 pad 8: Net-(C76-Pad2) -> Net-(C76-Pad1)
Routing:
- net -15V: track 0.00 -> 18.3 mm
- net Net-(R135-Pad1): track 0.00 -> 14.6 mm
- net Net-(RV1-Pad3): track 0.00 -> 12.2 mm, vias 0 -> 2
- net Net-(C50-Pad1): track 0.00 -> 11.4 mm
- net +15V: track 0.00 -> 6.63 mm
- added copper zone on F.Cu, net Net-(C50-Pad2)
- added copper zone on F.Cu, net Net-(C57-Pad1)
- added copper zone on F.Cu, net Net-(R7-Pad2)
Other:
- net class +/-15v added: clearance 0.15, trace_width 0.6, via_dia 0.6, via_drill 0.4
