File: Hardware/LIGHT_CONN.sch (KiCad schematic (older format))
At the start: 43 parts, among them P10 -15V, P11 ~4, P18 RX7, P19 3.3V, P20 TX6, P21 1.8V, P22 PSU_CTL, P23 GND, P31 P1, P32 L1.8_1, P33 L3.3_1, P34 P2, P35 L1.8_2, P36 L3.3_2, P37 P3, P38 L1.8_3, P39 L3.3_3, P40 P4, P41 L1.8_4, P42 L3.3_4, P6 CONN_02X14, P7 ~2, P8 +15V, P9 ~3, U22 PCA9685BS

Commit message: Mounting holes added
Parts:
- P11: value ~4 -> ~3
- P18: value RX7 -> RX6
- P20: value TX6 -> TX5
- P7: value ~2 -> ~1
- P9: value ~3 -> ~2
Changed lines of the file:
@@
 P 7550 4700
 F 0 "P11" H 7550 4800 50  0000 C CNN
-F 1 "~4" V 7650 4700 50  0001 C CNN
+F 1 "~3" V 7650 4700 50  0001 C CNN
 F 2 "Pin_Headers:Pin_Header_Straight_1x01" H 7550 4700 50  0001 C CNN
 F 3 "" H 7550 4700 50  0000 C CNN
@@
 P 7550 4450
 F 0 "P9" H 7550 4550 50  0000 C CNN
-F 1 "~3" V 7650 4450 50  0001 C CNN
+F 1 "~2" V 7650 4450 50  0001 C CNN
 F 2 "Pin_Headers:Pin_Header_Straight_1x01" H 7550 4450 50  0001 C CNN
 F 3 "" H 7550 4450 50  0000 C CNN
@@
 P 7550 4200
 F 0 "P7" H 7550 4300 50  0000 C CNN
-F 1 "~2" V 7650 4200 50  0001 C CNN
+F 1 "~1" V 7650 4200 50  0001 C CNN
 F 2 "Pin_Headers:Pin_Header_Straight_1x01" H 7550 4200 50  0001 C CNN
 F 3 "" H 7550 4200 50  0000 C CNN
@@
 P 7550 4950
 F 0 "P20" H 7550 5050 50  0000 C CNN
-F 1 "TX6" V 7650 4950 50  0001 C CNN
+F 1 "TX5" V 7650 4950 50  0001 C CNN
 F 2 "Pin_Headers:Pin_Header_Straight_1x01" H 7550 4950 50  0001 C CNN
 F 3 "" H 7550 4950 50  0000 C CNN
@@
 P 7550 5200
 F 0 "P18" H 7550 5300 50  0000 C CNN
-F 1 "RX7" V 7650 5200 50  0001 C CNN
+F 1 "RX6" V 7650 5200 50  0001 C CNN
 F 2 "Pin_Headers:Pin_Header_Straight_1x01" H 7550 5200 50  0001 C CNN
 F 3 "" H 7550 5200 50  0000 C CNN
